File: Prototype/KiCad/VIA.kicad_sch (KiCad schematic)
At the start: 104 parts, among them J10 VIA, J14 USB_B_Micro, J15 BOOT SEL, J16 VGA, J17 SWD, J18 3V3, J19 +5V, J21 JOY_POTS, J23 JOY_PORT, J4 KEYBOARD, J5 MOTOR, J6 9VAC, J7 DIN-6, U15 74LVC1G06, U17 74LVC1G06, U19 74LVC1G06, U20 MCP23S17_SO, U21 MCP23S17_SO, U22 TLV74311PDBVR, U23 W25Q16JVSSIQ, U24 RP2350B-QFN80, U25 74CBTD3861, U26 74CBTD3861, U27 74CBTD3861, U28 TLV74333PDBVR, U7 6522 VIA, U8 6522 VIA, Y2 12MHz

Commit message: - Updated to KiCad 10
Parts:
- X1, X2: value ~ -> (none)
Connections:
- net GND: now also J14.SH (Shield), J16.SH; no longer J14.6 (Shield), J16.0
