File: Prototype/KiCad/Vic20_2025_SMD.kicad_pcb (KiCad board)
At the start: 2 copper layers, 300 x 100 mm, 341 parts, among them J1 +5V, J10 VIA, J11 EDGE, J12 VIC, J13 USB_B_Micro, J14 USB_B_Micro, J15 BOOT SEL, J16 VGA, J17 SWD, J18 3V3, J19 +5V, J2 SWD, J20 VIC, J201 USB_B_Micro, J202 BOOT SEL, J203 Vic20 Cartridge Connector, J204 VGA, J205 SWD, J206 EDGE, J207 +5V, J21 JOY_POTS, J22 Spare, J23 JOY_PORT, J24 3v3, J25 SYNC, J3 SS-53000-001, J4 KEYBOARD, J5 MOTOR, J6 9VAC, J7 DIN-6, J8 DIN-5_180degree, J9 2350 BOOT SEL, Q1 BSS138, Q2 2SC2712-GR,LF, Q3 BSS138, U1 LD1117S33TR_SOT223, U10 74CBTD3861, U11 W25Q16JVSSIQ, U12 THS7316D, U13 TLV74311PDBVR, U14 RP2350A-QFN60, U15 74LVC1G06, U16 iCE40HX4K-TQ144, U17 74LVC1G06, U18 74LS245, U19 74LVC1G06, U2 MIC5504-1.2YM5, U20 MCP23S17_SO, U201 TLV74311PDBVR, U202 W25Q16JVSSIQ, U203 RP2350B-QFN80, U204 74LVC1G06, U205 74LVC245A, U206 IS6xC1024AL-xxH, U207 6502 CPU, U208 74LVC245A, U209 LD1117S33TR_SOT223, U21 MCP23S17_SO, U210 74LS245, U211 74CBTD3861, U22 TLV74311PDBVR, U23 W25Q16JVSSIQ, U24 RP2350B-QFN80, U25 74CBTD3861, U26 74CBTD3861, U27 74CBTD3861, U28 TLV74333PDBVR, U29 74CBTD3861, U3 W25Q16JVSSIQ, U30 74CBTD3861, U32 LM1881, U4 74LS245, U5 6561 VIC, U6 74CBTD3861, U7 6522 VIA, U8 6522 VIA, U9 74CBTD3861, Y1 12MHz, Y2 12MHz, Y201 12MHz

Commit message: - Updated to KiCad 10
Parts:
- D201: footprint Diode_SMD:D_SOD-123 -> Diode_SMD:D_SMA
- Q2: footprint Package_TO_SOT_SMD:SOT-23 -> Package_TO_SOT_SMD:TSOT-23
- U5: footprint Dave Footprints:DIP-40_6561 -> Package_DIP:DIP-40_W15.24mm_LongPads
Connections:
- net Net-(J25-Pin_2) renamed /Video FPGA/VSOUT
- net Net-(J25-Pin_3) renamed /Video FPGA/BPOUT
Routing:
- net GND: track 390.9 -> 397.1 mm
