File: Prototype/KiCad/VideoFPGA.kicad_sch (KiCad schematic)
At the start: 162 parts, among them J1 +5V, J11 EDGE, J12 VIC, J13 USB_B_Micro, J2 SWD, J20 VIC, J22 Spare, J24 3v3, J25 SYNC, J3 SS-53000-001, J8 DIN-5_180degree, J9 2350 BOOT SEL, Q1 BSS138, Q2 2SC2712-GR,LF, Q3 BSS138, U1 LD1117S33TR_SOT223, U10 74CBTD3861, U11 W25Q16JVSSIQ, U12 THS7316D, U13 TLV74311PDBVR, U14 RP2350A-QFN60, U16 iCE40HX4K-TQ144, U18 74LS245, U2 MIC5504-1.2YM5, U29 74CBTD3861, U3 W25Q16JVSSIQ, U30 74CBTD3861, U32 LM1881, U4 74LS245, U5 6561 VIC, U6 74CBTD3861, U9 74CBTD3861, Y1 12MHz

Commit message: - Updated to KiCad 10
Parts:
- Q2: footprint Package_TO_SOT_SMD:SOT-23 -> Package_TO_SOT_SMD:TSOT-23
- U5: footprint Dave Footprints:DIP-40_6561 -> Package_DIP:DIP-40_W15.24mm_LongPads
Connections:
- net GND: now also J13.SH (Shield); no longer J13.6 (Shield)
Other:
- moved on the sheet: C26, R18
