File: Prototype/Revision1/6502_6560/CPU_ROM.kicad_sch (KiCad schematic)
At the start: 75 parts, among them J201 USB_B_Micro, J202 BOOT SEL, J203 Vic20 Cartridge Connector, J204 VGA, J205 SWD, J206 EDGE, J207 +5V, U201 TLV74311PDBVR, U202 W25Q16JVSSIQ, U203 RP2350B-QFN80, U204 74LVC1G06, U205 74LVC245A, U206 IS6xC1024AL-xxH, U207 6502 CPU, U208 74LVC245A, U209 LD1117S33TR_SOT223, U210 74LS245, U211 74CBTD3861, Y201 12MHz

Commit message: - Initial component placement for protype 2, no routing done yet.
Parts:
- J201: footprint Dave Footprints:USB_Micro-B_Amphenol_10103594-0001LF_Horizontal -> _Custom:USB_Micro-B_Amphenol_10103594-0001LF_Horizontal
- J203: footprint SamacSys_Parts:307044558201 -> _Custom:Vic20-Cartridge-Connector; symbol SamacSys_Parts:307-044-558-201 -> _Custom:Vic20_Cartridge_Connector
- J204: footprint SamacSys_Parts:117345301 -> _Custom:DSUB-15
- Power201: footprint SamacSys_Parts:LEDC2012X90N -> LED_SMD:LED_0805_2012Metric
- U202: footprint Dave Footprints:SOIC-8_5.23x5.23mm_P1.27mm -> Package_SO:SOIC-8_5.3x5.3mm_P1.27mm
- U207: footprint Dave Footprints:DIP-40_6502 -> _Custom:DIP-40_6502
Changed lines of the file:
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@@
 			)
 		)
-		(property "Footprint" "Dave Footprints:DIP-40_6502"
+		(property "Footprint" "_Custom:DIP-40_6502"
 			(at 567.69 379.984 0)
 			(hide yes)
@@
 	)
 	(symbol
-		(lib_id "SamacSys_Parts:307-044-558-201")
+		(lib_id "_Custom:Vic20_Cartridge_Connector")
 		(at 589.28 398.78 0)
 		(mirror y)
@@
 			)
 		)
-		(property "Footprint" "SamacSys_Parts:307044558201"
-			(at 567.69 493.7 0)
+		(property "Footprint" "_Custom:Vic20-Cartridge-Connector"
+			(at 597.154 435.102 0)
 			(hide yes)
 			(show_name no)
@@
 		)
 		(property "Description" "Vic20 Cartridge Connector"
-			(at 589.28 398.78 0)
+			(at 589.026 398.526 90)
 			(hide yes)
 			(show_name no)
@@
 			)
 		)
-		(property "Footprint" "Dave Footprints:SOIC-8_5.23x5.23mm_P1.27mm"
+		(property "Footprint" "Package_SO:SOIC-8_5.3x5.3mm_P1.27mm"
 			(at 110.998 207.01 0)
 			(hide yes)
@@
 			)
 		)
-		(property "Footprint" "SamacSys_Parts:117345301"
+		(property "Footprint" "_Custom:DSUB-15"
 			(at 394.97 162.56 0)
 			(hide yes)
@@
 			)
 		)
-		(property "Footprint" "SamacSys_Parts:LEDC2012X90N"
+		(property "Footprint" "LED_SMD:LED_0805_2012Metric"
 			(at 114.3 345.44 0)
 			(hide yes)
@@
 			)
 		)
-		(property "Footprint" "Dave Footprints:USB_Micro-B_Amphenol_10103594-0001LF_Horizontal"
+		(property "Footprint" "_Custom:USB_Micro-B_Amphenol_10103594-0001LF_Horizontal"
 			(at 339.09 143.51 0)
 			(hide yes)
