File: Prototype/Revision1/6502_6560/Vic20_2025_SMD.kicad_pcb (KiCad board)
At the start: 2 copper layers, 300 x 100 mm, 341 parts, among them J1 +5V, J10 VIA, J11 EDGE, J12 VIC, J13 USB_B_Micro, J14 USB_B_Micro, J15 BOOT SEL, J16 VGA, J17 SWD, J18 3V3, J19 +5V, J2 SWD, J20 VIC, J201 USB_B_Micro, J202 BOOT SEL, J203 Vic20 Cartridge Connector, J204 VGA, J205 SWD, J206 EDGE, J207 +5V, J21 JOY_POTS, J22 Spare, J23 JOY_PORT, J24 3v3, J25 SYNC, J3 SS-53000-001, J4 KEYBOARD, J5 MOTOR, J6 9VAC, J7 DIN-6, J8 DIN-5_180degree, J9 2350 BOOT SEL, Q1 BSS138, Q2 2SC2712-GR,LF, Q3 BSS138, U1 LD1117S33TR_SOT223, U10 74CBTD3861, U11 W25Q16JVSSIQ, U12 THS7316D, U13 TLV74311PDBVR, U14 RP2350A-QFN60, U15 74LVC1G06, U16 iCE40HX4K-TQ144, U17 74LVC1G06, U18 74LS245, U19 74LVC1G06, U2 MIC5504-1.2YM5, U20 MCP23S17_SO, U201 TLV74311PDBVR, U202 W25Q16JVSSIQ, U203 RP2350B-QFN80, U204 74LVC1G06, U205 74LVC245A, U206 IS6xC1024AL-xxH, U207 6502 CPU, U208 74LVC245A, U209 LD1117S33TR_SOT223, U21 MCP23S17_SO, U210 74LS245, U211 74CBTD3861, U22 TLV74311PDBVR, U23 W25Q16JVSSIQ, U24 RP2350B-QFN80, U25 74CBTD3861, U26 74CBTD3861, U27 74CBTD3861, U28 TLV74333PDBVR, U29 74CBTD3861, U3 W25Q16JVSSIQ, U30 74CBTD3861, U32 LM1881, U4 74LS245, U5 6561 VIC, U6 74CBTD3861, U7 6522 VIA, U8 6522 VIA, U9 74CBTD3861, Y1 12MHz, Y2 12MHz, Y201 12MHz

Commit message: - Initial component placement for protype 2, no routing done yet.
Parts:
- removed C28, C35, C49, C50, C51, C52, C53, C54, C55, C58, C59, C60, C61, C62, C63, C67, C68, C69, C70, C71, C72, C74, C77, C78, C79: 100nf, Capacitor_SMD:C_0603_1608Metric
- removed C56, C57, C73, C80: 4.7uf, Capacitor_SMD:C_0805_2012Metric
- removed C75, C76: 8pf, Capacitor_SMD:C_0603_1608Metric
- removed C81: 470uf, Capacitor_THT:CP_Radial_D5.0mm_P2.50mm
- removed C83, C84: 1nf, Capacitor_SMD:C_0603_1608Metric
- removed D3: B140-E3, Diode_SMD:D_SOD-123
- removed FB1, FB2, FB3: FerriteBead_Small, Resistor_SMD:R_0805_2012Metric
- removed J10: VIA, Connector_PinHeader_2.54mm:PinHeader_1x20_P2.54mm_Vertical
- removed J14: USB_B_Micro, Dave Footprints:USB_Micro-B_Amphenol_10103594-0001LF_Horizontal
- removed J15: BOOT SEL, Connector_PinHeader_2.54mm:PinHeader_1x02_P2.54mm_Vertical
- removed J16: VGA, SamacSys_Parts:117345301
- removed J17: SWD, Connector_PinHeader_2.54mm:PinHeader_1x03_P2.54mm_Vertical
- removed J18: 3V3, Connector_PinHeader_2.54mm:PinHeader_1x03_P2.54mm_Vertical
- removed J19: +5V, Connector_PinHeader_2.54mm:PinHeader_2x04_P2.54mm_Vertical
- removed J21: JOY_POTS, Connector_PinHeader_2.54mm:PinHeader_1x03_P2.54mm_Vertical
- removed J23: JOY_PORT, Dave Footprints:JOYPORT_9PIN_HEADER
- removed J4: KEYBOARD, Dave Footprints:KEYBOARD_CON
- removed J5: MOTOR, Connector_PinHeader_2.54mm:PinHeader_1x02_P2.54mm_Vertical
- removed J6: 9VAC, Connector_PinHeader_2.54mm:PinHeader_1x02_P2.54mm_Vertical
- removed J7: DIN-6, Dave Footprints:SERIAL_CON_DIN6
- removed JP2: SolderJumper_2_Bridged, Jumper:SolderJumper-2_P1.3mm_Bridged2Bar_RoundedPad1.0x1.5mm
- removed Power2: POWER, SamacSys_Parts:LEDC2012X90N
- removed R38, R42, R44, R45, R46, R47, R48, R49, R50, R54, R60, R61, R63, R64, R66, R67, R69, R72: 10k, Resistor_SMD:R_0603_1608Metric
- removed R39, R40, R41, R55, R59, R73: 1k, Resistor_SMD:R_0603_1608Metric
- removed R51, R52, R53: 27R, Resistor_SMD:R_0603_1608Metric
- removed R56, R57, R58: 340, Resistor_SMD:R_0603_1608Metric
- removed TP10, TP11, TP8, TP9: TestPoint, TestPoint:TestPoint_Pad_1.0x1.0mm
- removed U15, U17, U19: 74LVC1G06, Package_TO_SOT_SMD:SOT-353_SC-70-5
- removed U20, U21: MCP23S17_SO, Package_SO:SOIC-28W_7.5x17.9mm_P1.27mm
- removed U22: TLV74311PDBVR, Package_TO_SOT_SMD:SOT-23-5
- removed U23: W25Q16JVSSIQ, Dave Footprints:SOIC-8_5.23x5.23mm_P1.27mm
- removed U24: RP2350B-QFN80, RP2350_KiCad-main:RP2350B_QFN-80_EP_10.573x10.573_Pitch0.4mm
- removed U25, U26, U27: 74CBTD3861, Package_SO:SSOP-24_3.9x8.7mm_P0.635mm
- removed U28: TLV74333PDBVR, Package_TO_SOT_SMD:SOT-23-5
- removed U7, U8: 6522 VIA, Dave Footprints:DIP-40_6522
- removed X1: ~, Dave Footprints:EDGE_CON_12P_TAPE
- removed X2: ~, Dave Footprints:EDGE_CON_24P
- removed Y2: 12MHz, Crystal:Crystal_SMD_SeikoEpson_FA238V-4Pin_3.2x2.5mm
- CDone1, Power1, Power201: footprint SamacSys_Parts:LEDC2012X90N -> LED_SMD:LED_0805_2012Metric
- J13, J201: footprint Dave Footprints:USB_Micro-B_Amphenol_10103594-0001LF_Horizontal -> _Custom:USB_Micro-B_Amphenol_10103594-0001LF_Horizontal
- J203: footprint SamacSys_Parts:307044558201 -> _Custom:Vic20-Cartridge-Connector
- J204: footprint SamacSys_Parts:117345301 -> _Custom:DSUB-15
- U11, U202, U3: footprint Dave Footprints:SOIC-8_5.23x5.23mm_P1.27mm -> Package_SO:SOIC-8_5.3x5.3mm_P1.27mm
- U207: footprint Dave Footprints:DIP-40_6502 -> _Custom:DIP-40_6502
Connections:
- net /BD0 renamed /CPU and ROM/BD0
- net /BD1 renamed /CPU and ROM/BD1
- net /BD2 renamed /CPU and ROM/BD2
- net /BD3 renamed /CPU and ROM/BD3
- net /BD4 renamed /CPU and ROM/BD4
- net /BD5 renamed /CPU and ROM/BD5
- net /BD6 renamed /CPU and ROM/BD6
- net /BD7 renamed /CPU and ROM/BD7
- net /CA0 renamed /CPU and ROM/CA0
- net /CA1 renamed /CPU and ROM/CA1
- net /CA10 renamed /CPU and ROM/CA10
- net /CA11 renamed /CPU and ROM/CA11
- net /CA12 renamed /CPU and ROM/CA12
- net /CA13 renamed /CPU and ROM/CA13
- net /CA14 renamed /CPU and ROM/CA14
- net /CA15 renamed /CPU and ROM/CA15
- net /CA2 renamed /CPU and ROM/CA2
- net /CA3 renamed /CPU and ROM/CA3
- net /CA4 renamed /CPU and ROM/CA4
- net /CA5 renamed /CPU and ROM/CA5
- net /CA6 renamed /CPU and ROM/CA6
- net /CA7 renamed /CPU and ROM/CA7
- net /CA8 renamed /CPU and ROM/CA8
- net /CA9 renamed /CPU and ROM/CA9
Routing:
- net /VIA/+5V0_RAIL_VIA: track 404.6 -> 0.00 mm, vias 12 -> 0
- net /VIA/~{RES}: track 198.3 -> 0.00 mm, vias 3 -> 0
- net /VIA/CA5: track 161.7 -> 0.00 mm, vias 3 -> 0
- net /VIA/~{NMI}: track 151.8 -> 0.00 mm, vias 1 -> 0
- net /VIA/~{IRQ}: track 146.7 -> 0.00 mm, vias 3 -> 0
- net /VIA/CA4: track 146.0 -> 0.00 mm, vias 1 -> 0
- net GND: track 397.1 -> 251.3 mm, vias 261 -> 166
- net /VIA/RESTORE: track 142.9 -> 0.00 mm, vias 2 -> 0
- net /VIA/CR/~{W}: track 139.4 -> 0.00 mm, vias 2 -> 0
- net /VIA/+3V3_RAIL_VIA: track 138.2 -> 0.00 mm, vias 13 -> 0
- net /VIA/CASS_MOTOR: track 132.5 -> 0.00 mm, vias 2 -> 0
- net /VIA/CASSETTE_SWITCH: track 129.8 -> 0.00 mm, vias 3 -> 0
- net /VIA/JOY0: track 125.1 -> 0.00 mm, vias 4 -> 0
- net /VIA/JOY1: track 122.9 -> 0.00 mm, vias 2 -> 0
- net /VIA/JOY2: track 122.1 -> 0.00 mm, vias 2 -> 0
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Other:
- board size 300 x 100 mm -> 199.8 x 100 mm
- board text removed: "I/O Board - Rev A - Dave Gaunt."
