File: Prototype/Revision1/6502_6560/VideoFPGA.kicad_sch (KiCad schematic)
At the start: 162 parts, among them J1 +5V, J11 EDGE, J12 VIC, J13 USB_B_Micro, J2 SWD, J20 VIC, J22 Spare, J24 3v3, J25 SYNC, J3 SS-53000-001, J8 DIN-5_180degree, J9 2350 BOOT SEL, Q1 BSS138, Q2 2SC2712-GR,LF, Q3 BSS138, U1 LD1117S33TR_SOT223, U10 74CBTD3861, U11 W25Q16JVSSIQ, U12 THS7316D, U13 TLV74311PDBVR, U14 RP2350A-QFN60, U16 iCE40HX4K-TQ144, U18 74LS245, U2 MIC5504-1.2YM5, U29 74CBTD3861, U3 W25Q16JVSSIQ, U30 74CBTD3861, U32 LM1881, U4 74LS245, U5 6561 VIC, U6 74CBTD3861, U9 74CBTD3861, Y1 12MHz

Commit message: - Initial component placement for protype 2, no routing done yet.
Parts:
- CDone1, Power1: footprint SamacSys_Parts:LEDC2012X90N -> LED_SMD:LED_0805_2012Metric
- J13: footprint Dave Footprints:USB_Micro-B_Amphenol_10103594-0001LF_Horizontal -> _Custom:USB_Micro-B_Amphenol_10103594-0001LF_Horizontal
- U11, U3: footprint Dave Footprints:SOIC-8_5.23x5.23mm_P1.27mm -> Package_SO:SOIC-8_5.3x5.3mm_P1.27mm
Changed lines of the file:
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@@
 			)
 		)
-		(property "Footprint" "Dave Footprints:SOIC-8_5.23x5.23mm_P1.27mm"
+		(property "Footprint" "Package_SO:SOIC-8_5.3x5.3mm_P1.27mm"
 			(at 80.518 191.77 0)
 			(hide yes)
@@
 			)
 		)
-		(property "Footprint" "SamacSys_Parts:LEDC2012X90N"
+		(property "Footprint" "LED_SMD:LED_0805_2012Metric"
 			(at 154.94 194.31 0)
 			(hide yes)
@@
 			)
 		)
-		(property "Footprint" "Dave Footprints:SOIC-8_5.23x5.23mm_P1.27mm"
+		(property "Footprint" "Package_SO:SOIC-8_5.3x5.3mm_P1.27mm"
 			(at 326.898 143.51 0)
 			(hide yes)
@@
 			)
 		)
-		(property "Footprint" "SamacSys_Parts:LEDC2012X90N"
+		(property "Footprint" "LED_SMD:LED_0805_2012Metric"
 			(at 43.18 58.42 0)
 			(hide yes)
@@
 			)
 		)
-		(property "Footprint" "Dave Footprints:USB_Micro-B_Amphenol_10103594-0001LF_Horizontal"
+		(property "Footprint" "_Custom:USB_Micro-B_Amphenol_10103594-0001LF_Horizontal"
 			(at 547.37 82.55 0)
 			(hide yes)
