File: Prototype/Revision2/VIC_CPU/Vic20_2025_SMD.kicad_sch (KiCad schematic)
At the start: 101 parts, among them J2 BOOT SEL, J3 SWD, J4 USB_B_Micro, J5 VGA, J6 Vic20 Cartridge Connector, J7 I/O Board Connector, J8 Audio / Video, J9 Frame Buffer, U1 W25Q16JVSSIQ, U10 IS6xC1024AL-xxH, U11 6502 CPU, U12 74CBTD3861, U13 74LVC245A, U14 74LVC245A, U3 RP2350B-QFN80, U4 iCE40HX4K-TQ144, U5 74CBTD3861, U6 6561 VIC, U7 74CBTD3861, U8 74CBTD3861, U9 74CBTD3861, Y1 12MHz

Commit message: - As the prototype currently spans 4 boards I have decided to spin a prototype revision 2 (two board prototype set) before i commit to the final layout and design.
Parts:
- removed C1: 100nf, Capacitor_SMD:C_0603_1608Metric, symbol Device:C_Small
- removed R1: 10k, Resistor_SMD:R_0603_1608Metric, symbol Device:R_Small
- removed U1: W25Q16JVSSIQ, Package_SO:SOIC-8_5.3x5.3mm_P1.27mm, symbol Dave:W25Q16JVSSIQ
- added C51: 100nf, Capacitor_SMD:C_0603_1608Metric, symbol Device:C_Small
- added C52: 4.7uf, Capacitor_SMD:C_0603_1608Metric, symbol Device:C_Small
- added J10: DM3D-SF, _Custom:DM3DSF_SDCard, symbol _Custom:DM3D-SF_SDCard
- added R41, R42, R43, R44, R45, R46, R47: 10k, Resistor_SMD:R_0603_1608Metric, symbol Device:R_Small
- J4: footprint Dave Footprints:USB_Micro-B_Amphenol_10103594-0001LF_Horizontal -> _Custom:USB_Micro-B_Amphenol_10103594-0001LF_Horizontal
- R2: value 1k -> 2k2
- U3: value RP2350B-QFN80 -> RP2354B-QFN80
Connections:
- net +3V3: now also C51.2, C52.2, J10.4 (VDD), R41.2, R42.2, R43.2, R44.2, R45.2, R46.2, R47.2
- net GND: now also C51.1, C52.1, J10.0 (GND), J10.6 (VSS), J10.B (SW_B)
- net 2350_QSPI.SCK: no longer names the net of U3.71 (QSPI_SCLK)
- net 2350_QSPI.SD0: no longer names the net of U3.72 (QSPI_SD0)
- net 2350_QSPI.SD1: no longer names the net of U3.74 (QSPI_SD1)
- net 2350_QSPI.SD2: no longer names the net of U3.73 (QSPI_SD2)
- net 2350_QSPI.SD3: no longer names the net of U3.70 (QSPI_SD3)
- new net: J10.8 (DAT1), R45.1
- new net: J10.1 (DAT2), R44.1
- new net: J10.A (SW_A), R47.1
- new net SPI1.RX: J10.7 (DAT0), R46.1
- new net SPI1.SCK: J10.5 (CLK), R41.1
- new net SPI1.TX: J10.3 (CMD), R42.1
- new net SPI1.~{CS}: J10.2 (CD/DAT3), R43.1
- no-connect marks 24 -> 29
Other:
- moved on the sheet: R2

Commit message: - Initial component placement for protype 2, no routing done yet.
Parts:
- J9: footprint Connector_PinSocket_2.54mm:PinSocket_2x10_P2.54mm_Vertical -> Connector_PinHeader_2.54mm:PinHeader_2x10_P2.54mm_Vertical
- U4: footprint SamacSys_Parts:QFP50P2200X2200X160-144N -> Package_QFP:LQFP-144_20x20mm_P0.5mm
Connections:
- net iCE40-SDI: now also U3.19 (GPIO19); no longer U3.20 (GPIO20)
- net iCE40-SDO: now also U3.20 (GPIO20); no longer U3.19 (GPIO19)
Changed lines of the file:
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@@
 		)
 	)
+	(global_label "iCE40-SDO"
+		(shape input)
+		(at 276.86 187.96 0)
+		(fields_autoplaced yes)
+		(effects
+			(font
+				(size 1.27 1.27)
+			)
+			(justify left)
+		)
+		(property "Intersheetrefs" "${INTERSHEET_REFS}"
+			(at 290.6704 187.96 0)
+			(hide yes)
+			(show_name no)
+			(do_not_autoplace no)
+			(effects
+				(font
+					(size 1.27 1.27)
+				)
+				(justify left)
+			)
+		)
+	)
 	(global_label "iCE40-CRESET"
 		(shape output)
@@
 		)
 	)
-	(global_label "iCE40-SDO"
-		(shape input)
-		(at 276.86 182.88 0)
-		(fields_autoplaced yes)
-		(effects
-			(font
-				(size 1.27 1.27)
-			)
-			(justify left)
-		)
-		(property "Intersheetrefs" "${INTERSHEET_REFS}"
-			(at 290.6704 182.88 0)
-			(hide yes)
-			(show_name no)
-			(do_not_autoplace no)
-			(effects
-				(font
-					(size 1.27 1.27)
-				)
-				(justify left)
-			)
-		)
-	)
 	(global_label "~{RESET}"
 		(shape input)
@@
 		)
 	)
-	(global_label "iCE40-SDI"
-		(shape output)
-		(at 276.86 187.96 0)
-		(fields_autoplaced yes)
-		(effects
-			(font
-				(size 1.27 1.27)
-			)
-			(justify left)
-		)
-		(property "Intersheetrefs" "${INTERSHEET_REFS}"
-			(at 289.9447 187.96 0)
-			(hide yes)
-			(show_name no)
-			(do_not_autoplace no)
-			(effects
-				(font
-					(size 1.27 1.27)
-				)
-				(justify left)
-			)
-		)
-	)
 	(global_label "~{NMI}"
 		(shape bidirectional)
@@
 		)
 	)
+	(global_label "iCE40-SDI"
+		(shape output)
+		(at 276.86 182.88 0)
+		(fields_autoplaced yes)
+		(effects
+			(font
+				(size 1.27 1.27)
+			)
+			(justify left)
+		)
+		(property "Intersheetrefs" "${INTERSHEET_REFS}"
+			(at 289.9447 182.88 0)
+			(hide yes)
+			(show_name no)
+			(do_not_autoplace no)
+			(effects
+				(font
+					(size 1.27 1.27)
+				)
+				(justify left)
+			)
+		)
+	)
 	(global_label "CPU_PHI2"
 		(shape output)
@@
 	)
 	(global_label "iCE40-SCK"
-		(shape bidirectional)
+		(shape output)
 		(at 276.86 177.8 0)
 		(fields_autoplaced yes)
@@
 		)
 		(property "Intersheetrefs" "${INTERSHEET_REFS}"
-			(at 291.7212 177.8 0)
+			(at 290.6099 177.8 0)
 			(hide yes)
 			(show_name no)
@@
 			)
 		)
-		(property "Footprint" "SamacSys_Parts:QFP50P2200X2200X160-144N"
+		(property "Footprint" "Package_QFP:LQFP-144_20x20mm_P0.5mm"
 			(at 536.448 330.454 0)
 			(hide yes)
@@
 			)
 		)
-		(property "Footprint" "Connector_PinSocket_2.54mm:PinSocket_2x10_P2.54mm_Vertical"
+		(property "Footprint" "Connector_PinHeader_2.54mm:PinHeader_2x10_P2.54mm_Vertical"
 			(at 269.24 452.12 0)
 			(hide yes)
@@
 			)
 		)
-		(property "Footprint" "SamacSys_Parts:QFP50P2200X2200X160-144N"
+		(property "Footprint" "Package_QFP:LQFP-144_20x20mm_P0.5mm"
 			(at 156.972 226.314 0)
 			(hide yes)
@@
 			)
 		)
-		(property "Footprint" "SamacSys_Parts:QFP50P2200X2200X160-144N"
+		(property "Footprint" "Package_QFP:LQFP-144_20x20mm_P0.5mm"
 			(at 604.012 259.334 0)
 			(hide yes)
@@
 			)
 		)
-		(property "Footprint" "SamacSys_Parts:QFP50P2200X2200X160-144N"
+		(property "Footprint" "Package_QFP:LQFP-144_20x20mm_P0.5mm"
 			(at 156.972 335.534 0)
 			(hide yes)

Commit message: - Added the prototype rev2 IO Board schematic.
Parts:
- CON6: renamed from J6; footprint _Custom:Vic20-Cartridge-Connector -> _Custom:CON_VIC20-CART; symbol _Custom:Vic20_Cartridge_Connector -> _Custom:CON_CART-Vic20
- SD10: renamed from J10; footprint _Custom:DM3DSF_SDCard -> _Custom:SDCARD_DM3DSF; symbol _Custom:DM3D-SF_SDCard -> _Custom:SDCARD_DM3D-SF
- U11: symbol Dave:6502_Pin_Order -> _Custom:6502_Pin_Order
- U13, U14: symbol Dave:74LVC245A -> _Custom:74LVC245A
- U4: symbol Dave:iCE40HX4K-TQ144 -> _Custom:iCE40HX4K-TQ144
- U6: symbol Dave:6561_VIC_Pin_Order -> _Custom:6561_VIC_Pin_Order
Changed lines of the file:
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@@
 	)
 	(symbol
-		(lib_id "_Custom:Vic20_Cartridge_Connector")
+		(lib_id "_Custom:CON_CART-Vic20")
 		(at 579.12 281.94 0)
 		(mirror y)
@@
 		(in_pos_files yes)
 		(dnp no)
-		(property "Reference" "J6"
-			(at 566.42 274.32 0)
-			(hide yes)
+		(property "Reference" "CON6"
+			(at 587.502 244.348 0)
 			(show_name no)
 			(do_not_autoplace no)
@@
 					(size 1.27 1.27)
 				)
+				(justify left top)
 			)
 		)
@@
 			)
 		)
-		(property "Footprint" "_Custom:Vic20-Cartridge-Connector"
+		(property "Footprint" "_Custom:CON_VIC20-CART"
 			(at 586.994 318.262 0)
 			(hide yes)
@@
 			(project "Vic20_2025_SMD"
 				(path "/8d9f0380-e2a9-4d9b-b9cb-48f88a6a36ba"
-					(reference "J6")
+					(reference "CON6")
 					(unit 1)
 				)
@@
 	)
 	(symbol
-		(lib_id "Dave:6502_Pin_Order")
+		(lib_id "_Custom:6502_Pin_Order")
 		(at 579.12 198.12 0)
 		(mirror y)
@@
 	)
 	(symbol
-		(lib_id "Dave:74LVC245A")
+		(lib_id "_Custom:74LVC245A")
 		(at 675.64 205.74 0)
 		(unit 1)
@@
 	)
 	(symbol
-		(lib_id "Dave:iCE40HX4K-TQ144")
+		(lib_id "_Custom:iCE40HX4K-TQ144")
 		(at 472.44 441.96 0)
 		(mirror y)
@@
 	)
 	(symbol
-		(lib_id "Dave:iCE40HX4K-TQ144")
+		(lib_id "_Custom:iCE40HX4K-TQ144")
 		(at 220.98 337.82 0)
 		(unit 3)
@@
 	)
 	(symbol
-		(lib_id "Dave:iCE40HX4K-TQ144")
+		(lib_id "_Custom:iCE40HX4K-TQ144")
 		(at 668.02 370.84 0)
 		(unit 2)
@@
 	)
 	(symbol
-		(lib_id "Dave:74LVC245A")
+		(lib_id "_Custom:74LVC245A")
 		(at 675.64 281.94 0)
 		(unit 1)
@@
 	)
 	(symbol
-		(lib_id "Dave:iCE40HX4K-TQ144")
+		(lib_id "_Custom:iCE40HX4K-TQ144")
 		(at 220.98 447.04 0)
 		(unit 4)
@@
 	)
 	(symbol
-		(lib_id "_Custom:DM3D-SF_SDCard")
+		(lib_id "_Custom:SDCARD_DM3D-SF")
 		(at 383.54 111.76 0)
 		(unit 1)
@@
 		(in_pos_files yes)
 		(dnp no)
-		(property "Reference" "J10"
-			(at 373.38 104.14 0)
-			(hide yes)
+		(property "Reference" "SD10"
+			(at 370.84 104.14 0)
 			(show_name no)
 			(do_not_autoplace no)
@@
 					(size 1.27 1.27)
 				)
+				(justify left top)
 			)
 		)
@@
 			)
 		)
-		(property "Footprint" "_Custom:DM3DSF_SDCard"
+		(property "Footprint" "_Custom:SDCARD_DM3DSF"
 			(at 412.75 206.68 0)
 			(hide yes)
@@
 			(project "Vic20_2025_SMD"
 				(path "/8d9f0380-e2a9-4d9b-b9cb-48f88a6a36ba"
-					(reference "J10")
+					(reference "SD10")
 					(unit 1)
 				)
@@
 	)
 	(symbol
-		(lib_id "Dave:6561_VIC_Pin_Order")
+		(lib_id "_Custom:6561_VIC_Pin_Order")
 		(at 375.92 325.12 0)
 		(mirror y)
