File: Prototype/Revision2/VIA_IO/VIA_IO.kicad_pcb (KiCad board)
At the start: 2 copper layers, 100 x 88.2 mm, 282 parts, among them CN1 CONTROL PORT, J1 +5V, J2 KEYBOARD, J3 AUDIO / VIDEO, J4 AV INPUT, J5 SWD, J7 DV INTERCONNECT, J8 HDMI, J9 IO BOARD INTERCONNECT, Q1 2SC2712-GR,LF, U1 iCE40HX1K-VQ100, U10 LM1881, U11 THS7316D, U12 TLV74311PDBVR, U13 RP2354A-QFN60, U14 74CBTD3861, U15 74CBTD3861, U16 MIC5504-1.2YM5, U2 TLV74333PDBVR, U3 LSF0108PW, U4 LSF0108PW, U5 LSF0108PW, U6 LSF0108PW, U7 LSF0108PW, U8 TXU0104PWR, U9 BD60GC0WEFJ-E2, Y1 12MHz

Commit message: - Routed the new prototype 2 IO board.
Parts:
- removed D2: ESDA6V1SC5, _Custom:SOT-553
- removed R102: 10k, Resistor_SMD:R_0603_1608Metric
- removed TP4: Composite, TestPoint:TestPoint_Pad_1.0x1.0mm
- added AC2: 9VAC, Connector_PinHeader_2.54mm:PinHeader_1x02_P2.54mm_Vertical, F.Cu at (87.2, 105.7)
- added C71: 4.7uf, Capacitor_SMD:C_0603_1608Metric, F.Cu at (71.1, 129.2)
- added D13: ESDALD05UG4X, Package_SON:USON-10_2.5x1.0mm_P0.5mm, F.Cu at (69.6, 135.1)
- added TP14: 9VAC_N, TestPoint:TestPoint_Pad_1.0x1.0mm, F.Cu at (153.1, 67.6)
- added TP15: 9VAC_L, TestPoint:TestPoint_Pad_1.0x1.0mm, F.Cu at (145.4, 67.6)
- C14, C15, C35, C54, C61, D4, D5, L1, R107, R108, R109, R110, R133, R47, R93, TP3, U12: moved to B.Cu
- C48, FB1, FB2, FB3, R101: moved to F.Cu
- JP1: value SolderJumper_2_Bridged -> CA2
- JP2: value SolderJumper_2_Bridged -> PA7
- JP3: value SolderJumper_2_Bridged -> PA0
- JP4: value SolderJumper_2_Bridged -> PA1
- TP1: value TestPoint -> GBIn7; moved to B.Cu
- TP2: value TestPoint -> GBin6; moved to B.Cu
- moved C14 67.7 mm to (152.8, 69.0), turned to 180 degrees
- moved C15 63.9 mm to (149.2, 64.5), turned to -90 degrees
- moved L1 59.4 mm to (149.2, 68.0), turned to 90 degrees
- moved C38 53.1 mm to (102.5, 98.7), turned to 180 degrees
- moved R95 49.5 mm to (98.1, 97.1)
- moved C41 44.2 mm to (93.8, 97.1), turned to 180 degrees
- moved TP8 40.1 mm to (92.9, 94.9), turned to 180 degrees
- moved TP7 39.9 mm to (93.1, 100.3), turned to 180 degrees
- moved C42 36.2 mm to (85.9, 100.1), turned to 180 degrees
- moved R96 34.5 mm to (81.4, 96.7), turned to 180 degrees
- moved C30 33.1 mm to (77.2, 116.7), turned to -90 degrees
- moved C40 32.6 mm to (81.5, 95.2)
- moved JP1 31.2 mm to (107.2, 120.5)
- moved TP9 29.7 mm to (76.0, 85.0), turned to 180 degrees
- moved TP10 29.1 mm to (81.4, 99.6), turned to 180 degrees
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Connections:
- BR1 pad 3: 9VAC22 -> /9VAC_N2
- BR1 pad 4: '9VAC22 -> /9VAC_L2
- D4 pad 1: /5V_9110.PA2 -> /5V_9110.PA4
- D4 pad 5: +5V -> /5V_9120.PB7
- D5 pad 1: /5V_9110.PA5 -> /5V_9110.PA2
- D5 pad 3: /5V_9120.PB7 -> +5V
- D5 pad 4: /5V_9110.PA4 -> /5V_9110.PA3
- D5 pad 5: /5V_9110.PA3 -> /5V_9110.PA5
- D9 pad 1: /SERIAL_ATTN_IO -> /5V_9120.CB1
- D9 pad 3: /5V_9120.CB1 -> /SERIAL_ATTN_IO
- D9 pad 4: /SERIAL_DATA_IO -> /SERIAL_CLK_IO
- D9 pad 5: /SERIAL_CLK_IO -> /SERIAL_DATA_IO
- DIN1 pad 4: Net-(DIN1-Pad4) -> Net-(C15-Pad2)
- DIN1 pad 5: Net-(DIN1-Pad4) -> Net-(C15-Pad2)
- DIN1 pad 6: Net-(DIN1-Pad6) -> /9VAC_L
- F1 pad 1: /'9VAC -> /9VAC_N
- R121 pad 1: /IO.IO0 -> /IO.CR_~{W}
- R121 pad 2: /3V3.IO0 -> /3V3.CR_~{W}
- R123 pad 1: /IO.CR_~{W} -> /IO.IO0
- R123 pad 2: /3V3.CR_~{W} -> /3V3.IO0
- U1 pad 62: /3V3.SO2 -> CLK_25MHZ
- U1 pad 63: CLK_25MHZ -> /3V3.SO2
- U1 pad 89: /3V3.CR_~{W} -> /3V3.IO0
- U1 pad 90: /3V3.IO0 -> /3V3.CR_~{W}
- U14 pad 2: /IO.CR_~{W} -> /IO.IO0
- U14 pad 21: /3V3.IO0 -> /3V3.CR_~{W}
- U14 pad 22: /3V3.CR_~{W} -> /3V3.IO0
- U14 pad 3: /IO.IO0 -> /IO.CR_~{W}
Routing:
- net +5V: track 132.5 -> 458.9 mm, vias 29 -> 39
- net /~{5V_RESET}: track 8.18 -> 185.1 mm, vias 0 -> 5
- net +3V3: track 295.3 -> 430.7 mm, vias 61 -> 74
- net /5V_9120.PB3: track 14.8 -> 132.6 mm, vias 1 -> 3
- net /iCE40.DONE: track 0.00 -> 104.1 mm, vias 0 -> 6
- net /SERIAL_ATTN_IN: track 6.55 -> 107.7 mm
- net /5V_9110.PA5: track 18.2 -> 119.2 mm, vias 0 -> 4
- net /CASSETTE_READ: track 14.1 -> 105.7 mm, vias 1 -> 3
- net CLK_25MHZ: track 2.20 -> 88.0 mm, vias 1 -> 2
- net /iCE40.~{RESET}: track 0.00 -> 85.0 mm, vias 0 -> 2
- net /5V_9120.PB7: track 2.52 -> 82.2 mm, vias 0 -> 3
- net GND: track 163.5 -> 242.5 mm, vias 71 -> 272
- net /5V_9110.PA4: track 17.6 -> 96.6 mm, vias 0 -> 1
- net /EXT_AUDIO_IN: track 0.00 -> 78.8 mm, vias 0 -> 1
- net /5V_9110.PA3: track 20.7 -> 98.8 mm, vias 0 -> 3
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Other:
- board text added: "I/O Board - Rev B - Dave Gaunt."
- board text removed: "I/O Board - Rev A - Dave Gaunt."
