File: Prototype/Revision2/VIA_IO/VIA_IO.kicad_sch (KiCad schematic)
At the start: 88 parts, among them CN8 CONTROL_PORT, J10 VIA, J12 VIC, J18 3V3, J19 +5V, J21 JOY_POTS, J22 JOY_POTS, J23 JOY_PORT, J24 JOY_PORT, J25 SYNC, J4 KEYBOARD, J5 MOTOR, J6 9VAC, J8 EDGE, SW1 POWER_SWITCH, U1 BD60GC0WEFJ-E2, U12 THS7316D, U15 74LVC1G06, U17 74LVC1G06, U18 74LVC1G06, U19 74LVC1G06, U28 TLV74333PDBVR, U32 LM1881, U7 6522 VIA, U8 6522 VIA

Commit message: - Added the prototype rev2 IO Board schematic.
Parts:
- removed C1: 2200uF, Capacitor_THT:CP_Radial_D10.0mm_P5.00mm, symbol Device:C_Polarized_Small
- removed C13, C8: 220nf, Capacitor_SMD:C_0805_2012Metric, symbol Device:C_Small
- removed C2: 100uF, Capacitor_THT:CP_Radial_D5.0mm_P2.50mm, symbol Device:C_Polarized_Small
- removed C80: 4.7uf, Capacitor_SMD:C_0603_1608Metric, symbol Device:C_Small
- removed C83, C84: 1nf, Capacitor_SMD:C_0603_1608Metric, symbol Device:C_Small
- removed CN8: CONTROL_PORT, _Custom:JOYPORT_DB9, symbol _Custom:CONTROL_PORT-C64
- removed D3: B140-E3, Diode_SMD:D_SOD-123, symbol Diode:B140-E3
- removed DIN3: DIN-6, _Custom:DIN-6, symbol Connector:DIN-6
- removed J12: VIC, Connector_PinHeader_2.54mm:PinHeader_1x03_P2.54mm_Vertical, symbol Connector:Conn_01x03_Pin
- removed J18: 3V3, Connector_PinHeader_2.54mm:PinHeader_1x03_P2.54mm_Vertical, symbol Connector:Conn_01x03_Pin
- removed J19: +5V, Connector_PinHeader_2.54mm:PinHeader_2x04_P2.54mm_Vertical, symbol Connector_Generic:Conn_02x04_Odd_Even
- removed J21, J22: JOY_POTS, Connector_PinHeader_2.54mm:PinHeader_1x03_P2.54mm_Vertical, symbol Connector:Conn_01x03_Pin
- removed J23, J24: JOY_PORT, Dave Footprints:JOYPORT_9PIN_HEADER, symbol Connector_Generic:Conn_02x05_Top_Bottom
- removed J25: SYNC, Connector_PinHeader_2.54mm:PinHeader_1x04_P2.54mm_Vertical, symbol Connector:Conn_01x04_Pin
- removed J4: KEYBOARD, _Custom:CON_VIC20_KEYBOARD, symbol _Custom:CON_Vic20_Keyboard
- removed J5: MOTOR, Connector_PinHeader_2.54mm:PinHeader_1x02_P2.54mm_Vertical, symbol Connector:Conn_01x02_Pin
- removed J6: 9VAC, Connector_PinHeader_2.54mm:PinHeader_1x02_P2.54mm_Vertical, symbol Connector:Conn_01x02_Pin
- removed J8: EDGE, Connector_PinHeader_2.54mm:PinHeader_1x03_P2.54mm_Vertical, symbol Connector_Generic:Conn_01x03
- removed JP3, JP4: SolderJumper_2_Bridged, Jumper:SolderJumper-2_P1.3mm_Open_RoundedPad1.0x1.5mm, symbol Jumper:SolderJumper_2_Open
- removed Power2: POWER, LED_SMD:LED_0805_2012Metric, symbol Device:LED_Filled
- removed U1: BD60GC0WEFJ-E2, Package_SO:HTSOP-8-1EP_3.9x4.9mm_P1.27mm_EP2.4x3.2mm, symbol _Custom:LDO_BD60GC0WEFJ-E2
- removed U15, U17, U18, U19: 74LVC1G06, Package_TO_SOT_SMD:SOT-353_SC-70-5, symbol 74xGxx:74LVC1G06
- removed U28: TLV74333PDBVR, Package_TO_SOT_SMD:SOT-23-5, symbol Regulator_Linear:MIC5504-1.2YM5
- removed U7, U8: 6522 VIA, _Custom:DIP-40_6522, symbol _Custom:6522_VIA_Pin_Order
- added C1, C16, C18, C19, C2, C20, C21, C22, C23, C24, C25, C26, C27, C29, C3, C31, C33, C45, C47, C48, C55, C57, C58, C59, C60, C61, C62, C63, C64, C65, C67, C69, C70, C71: 100nf, Capacitor_SMD:C_0603_1608Metric, symbol Device:C_Small
- added C13: 100uF, Capacitor_THT:CP_Radial_D5.0mm_P2.50mm, symbol Device:C_Polarized_Small
- added C14, C15: 220nf, Capacitor_SMD:C_0805_2012Metric, symbol Device:C_Small
- added C17, C46, C54, C66, C68: 4.7uf, Capacitor_SMD:C_0603_1608Metric, symbol Device:C_Small
- added C30, C32: 1nf, Capacitor_SMD:C_0603_1608Metric, symbol Device:C_Small
- added C43, C44: 10pf, Capacitor_SMD:C_0603_1608Metric, symbol Device:C_Small
- added C8: 2200uF, Capacitor_THT:CP_Radial_D10.0mm_P5.00mm, symbol Device:C_Polarized_Small
- added CDone1: DONE, LED_SMD:LED_0805_2012Metric, symbol Device:LED_Filled
- added CN1: CONTROL PORT, _Custom:JOYPORT_DB9, symbol _Custom:CONTROL_PORT-C64
- added D1: B140-E3, Diode_SMD:D_SOD-123, symbol Diode:B140-E3
- added D10: D_Dual_Series_ACK, Package_TO_SOT_SMD:SOT-23, symbol Device:D_Dual_Series_ACK
- added D2, D3, D4, D5, D6, D7, D8, D9: ESDA6V1SC5, _Custom:SOT-553, symbol Power_Protection:ESDA6V1SC5
- added DIN2: IEC SERIAL, _Custom:DIN-6, symbol Connector:DIN-6
- added J1: +5V, Connector_PinHeader_2.54mm:PinHeader_2x04_P2.54mm_Vertical, symbol Connector_Generic:Conn_02x04_Odd_Even
- added J2: JOY_POTS, Connector_PinHeader_2.54mm:PinHeader_1x03_P2.54mm_Vertical, symbol Connector:Conn_01x03_Pin
- added J3: KEYBOARD, _Custom:CON_VIC20_KEYBOARD, symbol _Custom:CON_Vic20_Keyboard
- added J4: AV INPUT, Connector_PinHeader_2.54mm:PinHeader_1x04_P2.54mm_Vertical, symbol Connector:Conn_01x04_Pin
- added J6: SWD, Connector_PinHeader_2.54mm:PinHeader_1x03_P2.54mm_Vertical, symbol Connector:Conn_01x03_Pin
- added J7: USB_B_Micro, _Custom:USB_Micro-B_Amphenol_10103594-0001LF_Horizontal, symbol Connector:USB_B_Micro
- added J8: DV INTERCONNECT, Connector_PinHeader_2.54mm:PinHeader_2x05_P2.54mm_Vertical, symbol Connector_Generic:Conn_02x05_Odd_Even
- added J9: HDMI, Connector_Video:HDMI_A_Amphenol_10029449-x01xLF_Horizontal, symbol Connector:HDMI_A
- added JP1, JP2, JP3, JP4: SolderJumper_2_Bridged, Jumper:SolderJumper-2_P1.3mm_Bridged_RoundedPad1.0x1.5mm, symbol Jumper:SolderJumper_2_Bridged
- added Je1: BOOT SEL, Connector_PinHeader_2.54mm:PinHeader_1x02_P2.54mm_Vertical, symbol Connector:Conn_01x02_Pin
- added Power1: POWER, LED_SMD:LED_0805_2012Metric, symbol Device:LED_Filled
- added Q1: 2SC2712-GR,LF, Package_TO_SOT_SMD:TSOT-23, symbol Transistor_BJT:2SC4213
- added R1, R101, R103, R104: 1k, Resistor_SMD:R_0603_1608Metric, symbol Device:R_Small
- added R10, R11, R12, R13, R14, R15, R16, R17, R18, R19, R20, R21, R22, R23, R24, R25, R26, R27, R28, R29, R3, R30, R31, R32, R33, R34, R35, R36, R37, R4, R5, R6, R7, R8, R9: 4k7, Resistor_SMD:R_0603_1608Metric, symbol Device:R_Small
- added R100, R112, R113, R114, R132, R133, R134, R135, R136, R137, R147, R47, R88, R97: 10k, Resistor_SMD:R_0603_1608Metric, symbol Device:R_Small
- added R102: 470, Resistor_SMD:R_0603_1608Metric, symbol Device:R_Small
- added R105, R106, R107, R108, R109, R110, R111, R148, R99: 27R, Resistor_SMD:R_0603_1608Metric, symbol Device:R_Small
- added R115, R116, R117, R118, R119, R120, R121, R122, R123, R124, R125, R126, R127, R128, R129, R130, R131: 0R, Resistor_SMD:R_0603_1608Metric, symbol Device:R_Small
- added R138, R48, R49, R50, R51, R52, R53, R54, R55, R56, R57, R58, R59, R60, R61, R62, R63, R64, R65, R66, R67, R68, R69, R70, R71, R72, R74, R75, R76, R77, R78, R79, R80, R81, R82, R83, R84, R85, R86, R87, R98: 2k2, Resistor_SMD:R_0603_1608Metric, symbol Device:R_Small
- added R139, R140, R141, R142, R143, R144, R145, R146: 220, Resistor_SMD:R_0603_1608Metric, symbol Device:R_Small
- added R42, R43, R44, R45, R46: 200k, Resistor_SMD:R_0603_1608Metric, symbol Device:R_Small
- added S1: RESET, Button_Switch_THT:SW_PUSH_6mm_H4.3mm, symbol Switch:SW_Push
- added TP1, TP11, TP12, TP13, TP2, TP3: TestPoint, TestPoint:TestPoint_Pad_1.0x1.0mm, symbol Connector:TestPoint
- added TP10: Luma, TestPoint:TestPoint_Pad_1.0x1.0mm, symbol Connector:TestPoint
- added TP4: Composite Sync, TestPoint:TestPoint_Pad_1.0x1.0mm, symbol Connector:TestPoint
- added TP5: Vertical Sync, TestPoint:TestPoint_Pad_1.0x1.0mm, symbol Connector:TestPoint
- added TP6: Horizontal Sync, TestPoint:TestPoint_Pad_1.0x1.0mm, symbol Connector:TestPoint
- added TP7: Odd / Even, TestPoint:TestPoint_Pad_1.0x1.0mm, symbol Connector:TestPoint
- added TP8: Composite, TestPoint:TestPoint_Pad_1.0x1.0mm, symbol Connector:TestPoint
- added TP9: Chroma, TestPoint:TestPoint_Pad_1.0x1.0mm, symbol Connector:TestPoint
- added U1: ICE40HX1K-VQ100, Package_QFP:LQFP-100_14x14mm_P0.5mm, symbol _Custom:ICE40HX1K-VQ100
- added U12: TLV74311PDBVR, Package_TO_SOT_SMD:SOT-23-5, symbol Regulator_Linear:MIC5504-1.2YM5
- added U13: RP2354A-QFN60, RP2350_KiCad-main:RP2350A_QFN-60_EP_7.75x7.75_Pitch0.4mm, symbol MCU_RaspberryPi_and_Boards:RP2350A-QFN60
- added U14, U15: ESDALD05UG4X, Package_SON:USON-10_2.5x1.0mm_P0.5mm, symbol Power_Protection:TPD4E02B04DQA
- added U16, U17: 74CBTD3861, Package_SO:SSOP-24_3.9x8.7mm_P0.635mm, symbol 74xx:74CBTD3861
- added U18: MIC5504-1.2YM5, Package_TO_SOT_SMD:SOT-23-5, symbol Regulator_Linear:MIC5504-1.2YM5
- added U2: TLV74333PDBVR, Package_TO_SOT_SMD:SOT-23-5, symbol Regulator_Linear:MIC5504-1.2YM5
- added U3, U4, U5, U6, U7: LSF0108PW, Package_SO:TSSOP-20_4.4x6.5mm_P0.65mm, symbol Logic_LevelTranslator:LSF0108PW
- added U8: TXU0104PWR, Package_SO:TSSOP-14_4.4x5mm_P0.65mm, symbol _Custom:TXU0104PWR
- added U9: BD60GC0WEFJ-E2, Package_SO:HTSOP-8-1EP_3.9x4.9mm_P1.27mm_EP2.4x3.2mm, symbol _Custom:LDO_BD60GC0WEFJ-E2
- added Y1: 12MHz, Crystal:Crystal_SMD_SeikoEpson_FA238V-4Pin_3.2x2.5mm, symbol Device:Crystal_GND24_Small
- C10, C9: value 1nf -> 220nf; footprint Capacitor_SMD:C_0603_1608Metric -> Capacitor_SMD:C_0805_2012Metric
- C11, C12: value 100nf -> 220nf; footprint Capacitor_SMD:C_0603_1608Metric -> Capacitor_SMD:C_0805_2012Metric
- C4, C5, C6, C7: value 220nf -> 100nf; footprint Capacitor_SMD:C_0805_2012Metric -> Capacitor_SMD:C_0603_1608Metric
- C51: value 100nf -> 10nf
- C52: value 100nf -> 1uf; footprint Capacitor_SMD:C_0603_1608Metric -> Capacitor_SMD:C_0805_2012Metric
- C56: value 4.7uf -> 100nf
- DIN1: value POWER_CON -> POWER
- EDGE2: value (none) -> USER PORT
- J10: value VIA -> IO BOARD INTERCONNECT
- J5: renamed from DIN2; value DIN-5_180degree -> AUDIO / VIDEO; footprint _Custom:DIN-5 -> (none)
- R2, R38: value 10k -> 4k7
- R39, R40, R41: value 1k -> 4k7
- R73: value 1k -> 2k2
- renumbered C40 to C34, C41 to C36, C42 to C37, C87 to C38, C82 to C39, C89 to C40, C88 to C41, C90 to C42, R3 to R89, R70 to R90, R71 to R91, R85 to R92, R84 to R93, R79 to R94, R78 to R95, R77 to R96, U12 to U10, U32 to U11
Connections:
- net MOTOR is gone; now on net MOTOR_6VDC: EDGE1.C,3 (CASS_MOTOR)
- net RESTORE is gone; now on net +3V3: R38.2
- net '9VAC~: now also C10.1, C9.2, EDGE2.11 (9V_AC_); no longer C4.1, C7.2
- net +3V3: now also C4.1, C5.1, C53.1, C6.1, C7.1, R2.2, R39.2, R40.2, R41.2, C1.1, C17.2, C18.2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
- net +5V: now also C35.1, R73.2, C13.1, C14.2, C24.2, C31.1, C63.2, C64.2, C68.2, CN1.7, D1.2 (A), D2.5 (K)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; no longer C12.2, C28.2, C35.2, C49.1, C50.1, C51.2, C52.2, C53.2, C6.2, R2.1, R38.1, R39.1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
- net 9VAC: now also C11.2
- net 9VAC~: now also C10.2, C12.1, EDGE2.10 (9V__AC); no longer C4.2, C5.1
- net Audio Out: now also C52.2
- net BPOUT: now also TP6.1, U13.36 (GPIO24)
- net COMP_COLOUR: now also J4.1 (Pin_1)
- net GND: now also C12.2, C35.2, C4.2, C49.1, C50.1, C53.2, C6.2, C7.2, C1.2, C13.2, C14.1, C15.1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; no longer C10.2, C11.1, C12.1, C35.1, C49.2, C50.2, C52.1, C53.1, C6.1, C7.1, R73.1
- net MOTOR_6VDC: now also U9.1 (VO), U9.2 (FB)
- net POT_X: now also C30.1, CN1.9, D3.4 (K), J2.1 (Pin_1); no longer C10.1
- net POT_Y: now also C32.1, CN1.5, D3.3 (K), J2.2 (Pin_2); no longer C9.2
- net SERIAL_ATTN_IN: now also JP2.2 (B); no longer R39.2
- net SYNC_LUMA: now also J4.2 (Pin_2)
- net VIC_COMPOSITE: now also U10.8 (CH.1_OUT); no longer U10.6 (CH.3_OUT)
- net VIC_LUMA: now also U10.6 (CH.3_OUT); no longer U10.8 (CH.1_OUT)
- net VSOUT: now also TP5.1, U13.37 (GPIO25)
- net '9VAC: now reaches F1.1, FL1.3
- net '9VAC: now also C11.1
- net at L1.2, SW1.4: now also C15.2
- net SERIAL_ATTN_IO: now reaches FB1.2
- net SERIAL_ATTN_IO: now also D9.3 (K), DIN2.3
- net SERIAL_CLK_IO: now reaches FB2.2
- net SERIAL_CLK_IO: now also D9.4 (K), DIN2.4
- net SERIAL_DATA_IO: now reaches FB3.2
- net SERIAL_DATA_IO: now also D9.5 (K), DIN2.5
- net +11.3V: now reaches BR1.1 (+)
- net +11.3V: now also C33.2, C8.1, U9.8 (VCC); no longer C11.2
- net at U10.1 (CH.1_IN): now also C37.1; no longer C34.1
- net at U10.3 (CH.3_IN): now also C34.1; no longer C37.1
- net at J5.4, J5.5, R94.2: now also TP8.1
- net at U11.1 (CSOUT): now also TP4.1
- net at U11.7 (OEOUT): now also TP7.1
- net at C42.2, R92.2: now also R96.2, TP10.1
- net at R95.2: now also TP9.1
- net BD0 renamed IO.DATA0
- net IO.DATA0: now also R124.1, U17.2 (A1)
- net BD1 renamed IO.DATA1
- net IO.DATA1: now also R125.1, U17.3 (A2)
- net BD2 renamed IO.DATA2
- net IO.DATA2: now also R126.1, U17.4 (A3)
- net BD3 renamed IO.DATA3
- net IO.DATA3: now also R127.1, U17.5 (A4)
- net BD4 renamed IO.DATA4
- net IO.DATA4: now also R128.1, U17.6 (A5)
- net BD5 renamed IO.DATA5
- net IO.DATA5: now also R129.1, U17.7 (A6)
- net BD6 renamed IO.DATA6
- net IO.DATA6: now also R130.1, U17.8 (A7)
- net BD7 renamed IO.DATA7
- net IO.DATA7: now also R131.1, U17.9 (A8)
- net CA0 renamed IO.ADDRESS0
- net IO.ADDRESS0: now also R115.1, U16.2 (A1)
- net CA1 renamed IO.ADDRESS1
- net IO.ADDRESS1: now also R116.1, U16.3 (A2)
- net CA2 renamed IO.ADDRESS2
- net IO.ADDRESS2: now also R117.1, U16.4 (A3)
- net CA3 renamed IO.ADDRESS3
- net IO.ADDRESS3: now also R118.1, U16.5 (A4)
- net CA4 renamed IO.ADDRESS4
- net IO.ADDRESS4: now also R119.1, U16.6 (A5)
- net CA5 renamed IO.ADDRESS5
- net IO.ADDRESS5: now also R120.1, U16.7 (A6)
- net CASSETTE_SWITCH renamed 5V_9110.PA6
- net 5V_9110.PA6: now also D2.1 (K), D5.5 (K), R49.1, U3.17 (B2)
- net CASS_READ renamed CASSETTE_READ
- net CB1 renamed 5V_9110.CB1
- net CB2 renamed 5V_9110.CB2
- net COL3/CASS_WRITE renamed 5V_9120.PB3
- net CR/~{W} renamed IO.CR_~{W}
- net IO0 renamed IO.IO0
- net JOY0 renamed 5V_9110.PA2
- net JOY1 renamed 5V_9110.PA3
- net JOY2 renamed 5V_9110.PA4
- net LIGHT_PEN renamed 5V_9110.PA5
- net PB0 renamed 5V_9110.PB0
- net PB1 renamed 5V_9110.PB1
- net PB2 renamed 5V_9110.PB2
- net PB3 renamed 5V_9110.PB3
- net PB4 renamed 5V_9110.PB4
- net PB5 renamed 5V_9110.PB5
- net PB6 renamed 5V_9110.PB6
- net PB7 renamed 5V_9110.PB7
- net SERIAL_CLK_IN renamed 5V_9120.CA2
- net SERIAL_DATA_IN renamed 5V_9120.CB2
- net SO2 renamed IO.SO2
- net ~{IRQ} renamed 5V_9120.~{IRQ}
- net ~{NMI} renamed 5V_9110.~{NMI}
- net ~{RES} renamed ~{5V_RESET}
- new net: R110.1, U13.15 (GPIO11)
- new net: R114.1, U17.13 (B10)
- new net: R113.1, U17.14 (B9)
- new net: R136.1, U17.23 (~{OE})
- new net: C29.2, R46.1, U7.19 (RefB), U7.20 (EN)
- new net: TP3.1, U8.10 (B4Y)
- new net: R47.1, U8.5 (A4)
- new net: C27.2, R44.1, U5.19 (RefB), U5.20 (EN)
- new net: C16.2, D1.1 (K), U2.1 (VIN), U2.3 (EN)
- new net: R97.2, S1.1, U13.26 (RUN)
- new net: R134.1, U17.10 (A9)
- new net: R135.1, U17.11 (A10)
- new net: R111.1, U13.33 (GPIO21)
- new net: TP12.1, U13.42 (GPIO28_ADC2)
- new net: C46.2, R99.2, U13.46 (VREG_AVDD)
- new net: C50.2, Q1.1 (B), R103.2, R104.1
- new net: R132.1, U16.11 (A10)
- new net: R112.1, U16.13 (B10)
- new net: R133.1, U16.23 (~{OE})
- new net: R106.1, U13.51 (USB_DM)
- new net: Power1.1 (K), R1.2
- new net: TP2.1, U1.15 (IOL_7A_GBIN6)
- new net: C43.2, U13.21 (XIN), Y1.1
- new net: C44.2, R101.1, Y1.3
- new net: C26.2, R43.1, U4.19 (RefB), U4.20 (EN)
- new net: C25.2, R42.1, U3.19 (RefB), U3.20 (EN)
- new net: CDone1.1 (K), R148.1
- new net: C52.1, Q1.2 (E), R102.2
- new net: D10.3 (K), U1.75 (VPP_2V5)
- new net: R105.1, U13.52 (USB_DP)
- new net: TP11.1, U13.41 (GPIO27_ADC1)
- new net: Je1.1 (Pin_1), R98.2
- new net: C28.2, R45.1, U6.19 (RefB), U6.20 (EN)
- new net: R108.1, U13.13 (GPIO9)
- new net: TP1.1, U1.13 (IOL_6B_GBIN7)
- new net: R109.1, U13.14 (GPIO10)
- new net: R101.2, U13.22 (XOUT)
- new net: R107.1, U13.12 (GPIO8)
- new net: TP13.1, U13.43 (GPIO29_ADC3)
- new net +1V1: C45.2, C47.2, C49.2, C54.2, U12.5 (VOUT), U13.23 (DVDD), U13.39 (DVDD), U13.6 (DVDD)
- new net +1V2: C66.2, C67.1, C69.1, C70.1, C71.1, U1.11 (VCC_1), U1.35 (VCC_2), U1.61 (VCC_3), U1.77 (VCC_4), U18.5 (VOUT)
- new net 2354_SWCLK: J6.1 (Pin_1), U13.24 (SWCLK)
- new net 2354_SWDIO: J6.3 (Pin_3), U13.25 (SWDIO)
- new net 2354_USB_D+: J7.3 (D+), R105.2
- new net 2354_USB_D-: J7.2 (D-), R106.2
- new net 3V3.ADDRESS0: R115.2, U1.78 (IOT_73), U16.22 (B1)
- new net 3V3.ADDRESS1: R116.2, U1.79 (IOT_74), U16.21 (B2)
- new net 3V3.ADDRESS2: R117.2, U1.80 (IOT_75), U16.20 (B3)
- new net 3V3.ADDRESS3: R118.2, U1.81 (IOT_77), U16.19 (B4)
- new net 3V3.ADDRESS4: R119.2, U1.82 (IOT_78), U16.18 (B5)
- new net 3V3.ADDRESS5: R120.2, U1.83 (IOT_79), U16.17 (B6)
- new net 3V3.CR_~{W}: R123.2, U1.89 (IOT_84_GBIN1), U16.14 (B9)
- new net 3V3.DATA0: R124.2, U1.85 (IOT_80), U17.22 (B1)
- new net 3V3.DATA1: R125.2, U1.86 (IOT_81), U17.21 (B2)
- new net 3V3.DATA2: R126.2, U1.87 (IOT_82), U17.20 (B3)
- new net 3V3.DATA3: R127.2, U1.91 (IOT_86), U17.19 (B4)
- new net 3V3.DATA4: R128.2, U1.93 (IOT_87), U17.18 (B5)
- new net 3V3.DATA5: R129.2, U1.94 (IOT_88), U17.17 (B6)
- new net 3V3.DATA6: R130.2, U1.95 (IOT_89), U17.16 (B7)
- new net 3V3.DATA7: R131.2, U1.96 (IOT_90), U17.15 (B8)
- new net 3V3.IO0: R122.2, U1.90 (IOT_85_GBIN0), U16.15 (B8)
- new net 3V3.SO2: R121.2, U1.62 (IOR_60_GBIN3), U16.16 (B7)
- new net 3V3_9110.CA1: U1.29 (IOB_29), U8.11 (B3Y)
- new net 3V3_9110.CA2: R18.1, U1.26 (IOB_26), U5.3 (A1)
- new net 3V3_9110.CB1: R19.1, U1.30 (IOB_30), U5.4 (A2)
- new net 3V3_9110.CB2: R20.1, U1.27 (IOB_27), U5.5 (A3)
- new net 3V3_9110.PA0: R9.1, U1.64 (IOR_63), U3.10 (A8)
- new net 3V3_9110.PA1: R8.1, U1.65 (IOR_64), U3.9 (A7)
- new net 3V3_9110.PA2: R7.1, U1.66 (IOR_65), U3.8 (A6)
- new net 3V3_9110.PA3: R6.1, U1.68 (IOR_67), U3.7 (A5)
- new net 3V3_9110.PA4: R5.1, U1.69 (IOR_68), U3.6 (A4)
- new net 3V3_9110.PA5: R4.1, U1.71 (IOR_69), U3.5 (A3)
- new net 3V3_9110.PA6: R3.1, U1.72 (IOR_70), U3.4 (A2)
- new net 3V3_9110.PA7: R2.1, U1.73 (IOR_71), U3.3 (A1)
- new net 3V3_9110.PB0: R17.1, U1.51 (IOR_52), U4.10 (A8)
- new net 3V3_9110.PB1: R16.1, U1.52 (IOR_53), U4.9 (A7)
- new net 3V3_9110.PB2: R15.1, U1.53 (IOR_54), U4.8 (A6)
- new net 3V3_9110.PB3: R14.1, U1.54 (IOR_55), U4.7 (A5)
- new net 3V3_9110.PB4: R13.1, U1.56 (IOR_56), U4.6 (A4)
- new net 3V3_9110.PB5: R12.1, U1.57 (IOR_57), U4.5 (A3)
- new net 3V3_9110.PB6: R11.1, U1.59 (IOR_58), U4.4 (A2)
- new net 3V3_9110.PB7: R10.1, U1.60 (IOR_59), U4.3 (A1)
- new net 3V3_9110.~{NMI}: R21.1, U1.28 (IOB_28), U5.6 (A4)
- new net 3V3_9120.CA1: U1.36 (IOB_34), U8.13 (B1Y)
- new net 3V3_9120.CA2: R22.1, U1.40 (IOB_41), U5.7 (A5)
- new net 3V3_9120.CB1: R23.1, U1.37 (IOB_37), U5.8 (A6)
- new net 3V3_9120.CB2: R24.1, U1.41 (IOB_42_CBSEL0), U5.9 (A7)
- new net 3V3_9120.PA0: R33.1, U1.1 (IOL_1A), U6.10 (A8)
- new net 3V3_9120.PA1: R32.1, U1.2 (IOL_1B), U6.9 (A7)
- new net 3V3_9120.PA2: R31.1, U1.3 (IOL_2A), U6.8 (A6)
- new net 3V3_9120.PA3: R30.1, U1.4 (IOL_2B), U6.7 (A5)
- new net 3V3_9120.PA4: R29.1, U1.7 (IOL_3A), U6.6 (A4)
- new net 3V3_9120.PA5: R28.1, U1.8 (IOL_3B), U6.5 (A3)
- new net 3V3_9120.PA6: R27.1, U1.9 (IOL_5A), U6.4 (A2)
- new net 3V3_9120.PA7: R26.1, U1.10 (IOL_5B), U6.3 (A1)
- new net 3V3_9120.PB0: R41.1, U1.12 (IOL_6A), U7.10 (A8)
- new net 3V3_9120.PB1: R40.1, U1.16 (IOL_7B), U7.9 (A7)
- new net 3V3_9120.PB2: R39.1, U1.18 (IOL_8A), U7.8 (A6)
- new net 3V3_9120.PB3: R38.1, U1.19 (IOL_8B), U7.7 (A5)
- new net 3V3_9120.PB4: R37.1, U1.20 (IOL_10A), U7.6 (A4)
- new net 3V3_9120.PB5: R36.1, U1.21 (IOL_10B), U7.5 (A3)
- new net 3V3_9120.PB6: R35.1, U1.24 (IOL_12A), U7.4 (A2)
- new net 3V3_9120.PB7: R34.1, U1.25 (IOL_12B), U7.3 (A1)
- new net 3V3_9120.~{IRQ}: R25.1, U1.42 (IOB_43_CBSEL1), U5.10 (A8)
- new net 5V_9110.CA2: JP1.1 (A), R64.1, U5.18 (B1)
- new net 5V_9110.PA0: JP3.1 (A), R55.1, U3.11 (B8)
- new net 5V_9110.PA1: JP4.1 (A), R54.1, U3.12 (B7)
- new net 5V_9110.PA7: JP2.1 (A), R48.1, U3.18 (B1)
- new net 5V_9120.CB1: D9.1 (K), DIN2.1, R69.1, U5.13 (B6)
- new net 5V_9120.PA0: J3.20 (Pin_20), R79.1, U6.11 (B8)
- new net 5V_9120.PA1: J3.19 (Pin_19), R78.1, U6.12 (B7)
- new net 5V_9120.PA2: J3.18 (Pin_18), R77.1, U6.13 (B6)
- new net 5V_9120.PA3: J3.17 (Pin_17), R76.1, U6.14 (B5)
- new net 5V_9120.PA4: J3.16 (Pin_16), R75.1, U6.15 (B4)
- new net 5V_9120.PA5: J3.15 (Pin_15), R74.1, U6.16 (B3)
- new net 5V_9120.PA6: J3.14 (Pin_14), R73.1, U6.17 (B2)
- new net 5V_9120.PA7: J3.13 (Pin_13), R72.1, U6.18 (B1)
- new net 5V_9120.PB0: J3.12 (Pin_12), R87.1, U7.11 (B8)
- new net 5V_9120.PB1: J3.11 (Pin_11), R86.1, U7.12 (B7)
- new net 5V_9120.PB2: J3.10 (Pin_10), R85.1, U7.13 (B6)
- new net 5V_9120.PB4: J3.8 (Pin_8), R83.1, U7.15 (B4)
- new net 5V_9120.PB5: J3.7 (Pin_7), R82.1, U7.16 (B3)
- new net 5V_9120.PB6: J3.6 (Pin_6), R81.1, U7.17 (B2)
- new net 5V_9120.PB7: CN1.4, D4.3 (K), J3.5 (Pin_5), R80.1, U7.18 (B1)
- new net CLK_25MHZ: R111.2, U1.63 (IOR_61_GBIN2)
- new net COMP_SOUND: C51.2, J4.3 (Pin_3), R103.1
- new net DVI_TX0+: J9.7 (D0+), R143.2, U15.5 (IO4), U15.6 (NC)
- new net DVI_TX0-: J9.9 (D0-), R144.2, U15.4 (IO3), U15.7 (NC)
- new net DVI_TX1+: J9.4 (D1+), R141.2, U14.2 (IO2), U14.9 (NC)
- new net DVI_TX1-: J9.6 (D1-), R142.2, U14.1 (IO1), U14.10 (NC)
- new net DVI_TX2+: J9.1 (D2+), R139.2, U14.5 (IO4), U14.6 (NC)
- new net DVI_TX2-: J9.3 (D2-), R140.2, U14.4 (IO3), U14.7 (NC)
- new net DVI_TXC+: J9.10 (CK+), R145.2, U15.2 (IO2), U15.9 (NC)
- new net DVI_TXC-: J9.12 (CK-), R146.2, U15.1 (IO1), U15.10 (NC)
- new net EXT_AUDIO_IN: J4.4 (Pin_4), R104.2
- new net HALF_DOT_CLOCK: J8.9 (Pin_9), U13.35 (GPIO23)
- new net LANE.0+: R143.1, U13.19 (GPIO15)
- new net LANE.0-: R144.1, U13.18 (GPIO14)
- new net LANE.1+: R141.1, U13.28 (GPIO17)
- new net LANE.1-: R142.1, U13.27 (GPIO16)
- new net LANE.2+: R139.1, U13.31 (GPIO19)
- new net LANE.2-: R140.1, U13.29 (GPIO18)
- new net LANE.C+: R145.1, U13.17 (GPIO13)
- new net LANE.C-: R146.1, U13.16 (GPIO12)
- new net MOTOR_ENABLE: JP1.2 (B), U9.5 (EN)
- new net PixelData0: J8.1 (Pin_1), U13.2 (GPIO0)
- new net PixelData1: J8.3 (Pin_3), U13.3 (GPIO1)
- new net PixelData2: J8.5 (Pin_5), U13.4 (GPIO2)
- new net PixelData3: J8.7 (Pin_7), U13.5 (GPIO3)
- new net PixelData4: J8.2 (Pin_2), U13.7 (GPIO4)
- new net PixelData5: J8.4 (Pin_4), U13.8 (GPIO5)
- new net PixelData6: J8.6 (Pin_6), U13.9 (GPIO6)
- new net PixelData7: J8.8 (Pin_8), U13.10 (GPIO7)
- new net RESTORE_KEY: J3.3 (Pin_3), R88.1, U8.4 (A3)
- new net iCE40.DONE: CDone1.2 (A), R138.2, U1.43 (CDONE), U13.34 (GPIO22)
- new net iCE40.SCK: R109.2, U1.48 (IOB_46_SCK)
- new net iCE40.SDI: R110.2, U1.46 (IOB_45_SDI)
- new net iCE40.SDO: R107.2, U1.45 (IOB_44_SDO)
- new net iCE40.~{RESET}: R137.2, U1.44 (CRESET_B), U13.32 (GPIO20)
- new net iCE40.~{SS}: R108.2, R147.2, U1.49 (IOB_47_SS)
- new net ~{3V3_RESET}: U1.33 (IOB_35_GBIN5), U13.40 (GPIO26_ADC0), U8.12 (B2Y)
- new net ~{CS}: R100.2, R98.1, U13.60 (QSPI_SS)
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Other:
- note added: "AUDIO / VIDEO"
- note added: "CASSETTE_WRITE / COL3"
- note added: "COL0"
- note added: "COL1"
- note added: "COL2"
- note added: "COL4"
- note added: "COL5"
- note added: "COL6"
- note added: "FIRE"
- note added: "FIRE_BUTTON/LIGHT_PEN"
- note added: "IEC SERIAL"
- note added: "J0/JOY_UP"
- note added: "J1/JOY_DOWN"
- note added: "J2/JOY_LEFT"
- note added: "J3 / JOY_RIGHT / COL7"
- note added: "J3/JOY_RIGHT / COL7"
- note added: "ROW0"
- note added: "ROW1"
- note added: "ROW2"
- note added: "ROW3"
- note added: "ROW4"
- note added: "ROW5"
- note added: "ROW6"
- note added: "ROW7"
- note added: "SERIAL_ATTN_OUT"
- note added: "SERIAL_CLK_IN"
- note added: "SERIAL_CLK_OUT"
- note added: "SERIAL_DATA_IN"
- note added: "SERIAL_DATA_OUT"
- note added: "SERIAL_SRQ_IN"
- note added: "TAPE"
- title: VIC 2025 -> VIC 2026 Prototype IO Board
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
Commit message: - Initial layout of all the major components.
Parts:
- removed C37, C62, C71: 100nf, Capacitor_SMD:C_0603_1608Metric, symbol Device:C_Small
- removed C66: 4.7uf, Capacitor_SMD:C_0603_1608Metric, symbol Device:C_Small
- removed D10: D_Dual_Series_ACK, Package_TO_SOT_SMD:SOT-23, symbol Device:D_Dual_Series_ACK
- removed D5, D6, D7, D8: ESDA6V1SC5, _Custom:SOT-553, symbol Power_Protection:ESDA6V1SC5
- removed J2: JOY_POTS, Connector_PinHeader_2.54mm:PinHeader_1x03_P2.54mm_Vertical, symbol Connector:Conn_01x03_Pin
- removed J4: AV INPUT, Connector_PinHeader_2.54mm:PinHeader_1x04_P2.54mm_Vertical, symbol Connector:Conn_01x04_Pin
- removed J5: AUDIO / VIDEO, symbol Connector:DIN-5_180degree
- removed J6: SWD, Connector_PinHeader_2.54mm:PinHeader_1x03_P2.54mm_Vertical, symbol Connector:Conn_01x03_Pin
- removed J7: USB_B_Micro, _Custom:USB_Micro-B_Amphenol_10103594-0001LF_Horizontal, symbol Connector:USB_B_Micro
- removed R114, R137: 10k, Resistor_SMD:R_0603_1608Metric, symbol Device:R_Small
- removed R138: 2k2, Resistor_SMD:R_0603_1608Metric, symbol Device:R_Small
- removed R90: 1K, Resistor_SMD:R_0603_1608Metric, symbol Device:R_Small
- removed U10: THS7316D, Package_SO:SO-8_3.9x4.9mm_P1.27mm, symbol _Custom:VIDEO_AMP_THS7316D
- removed U11: LM1881, Package_SO:SO-8_3.9x4.9mm_P1.27mm, symbol Video:LM1881
- removed U18: MIC5504-1.2YM5, Package_TO_SOT_SMD:SOT-23-5, symbol Regulator_Linear:MIC5504-1.2YM5
- added AC1: 9VAC, Connector_PinHeader_2.54mm:PinHeader_1x02_P2.54mm_Vertical, symbol Connector:Conn_01x02_Pin
- added C35: 10nf, Capacitor_SMD:C_0603_1608Metric, symbol Device:C_Small
- added C64, C68: 100nf, Capacitor_SMD:C_0603_1608Metric, symbol Device:C_Small
- added D12: D_Dual_Series_ACK, Package_TO_SOT_SMD:SOT-23, symbol Device:D_Dual_Series_ACK
- added D3, D6, D7, D8: ESDALD05UG4X, Package_SON:USON-10_2.5x1.0mm_P0.5mm, symbol Power_Protection:TPD4E02B04DQA
- added J3: AUDIO / VIDEO, _Custom:DIN-5, symbol Connector:DIN-5_180degree
- added J4: AV INPUT, Connector_PinHeader_2.54mm:PinHeader_1x08_P2.54mm_Vertical, symbol Connector:Conn_01x08_Pin
- added J5: SWD, Connector_PinHeader_2.54mm:PinHeader_1x03_P2.54mm_Vertical, symbol Connector:Conn_01x03_Pin
- added J6: USB_B_Micro, _Custom:USB_Micro-B_Amphenol_10103594-0001LF_Horizontal, symbol Connector:USB_B_Micro
- added R112, R132: 10k, Resistor_SMD:R_0603_1608Metric, symbol Device:R_Small
- added R133: 2k2, Resistor_SMD:R_0603_1608Metric, symbol Device:R_Small
- added R88: 470R, Resistor_SMD:R_0603_1608Metric, symbol Device:R_Small
- added U10: LM1881, Package_SO:SO-8_3.9x4.9mm_P1.27mm, symbol Video:LM1881
- added U11: THS7316D, Package_SO:SO-8_3.9x4.9mm_P1.27mm, symbol _Custom:VIDEO_AMP_THS7316D
- added U16: MIC5504-1.2YM5, Package_TO_SOT_SMD:SOT-23-5, symbol Regulator_Linear:MIC5504-1.2YM5
- C36: value 100nf -> 1uf; footprint Capacitor_SMD:C_0603_1608Metric -> Capacitor_SMD:C_0805_2012Metric
- C38: value 100nf -> 510pf
- C42: value 510pf -> 100nf
- C43: value 10pf -> 100nf
- C45: value 100nf -> 10pf
- C46: value 4.7uf -> 100nf
- C48, C65: value 100nf -> 4.7uf
- C51: value 10nf -> 100nf
- C52: value 1uf -> 100nf; footprint Capacitor_SMD:C_0805_2012Metric -> Capacitor_SMD:C_0603_1608Metric
- J1: footprint Connector_PinHeader_2.54mm:PinHeader_2x04_P2.54mm_Vertical -> Connector_PinHeader_2.54mm:PinHeader_2x03_P2.54mm_Vertical; symbol Connector_Generic:Conn_02x04_Odd_Even -> Connector_Generic:Conn_02x03_Odd_Even
- Je1, R105, R106, S1: now not fitted; now left out of the parts list
- R10, R11, R12, R13, R14, R15, R16, R17, R18, R19, R2, R20, R21, R22, R23, R24, R25, R26, R27, R28, R29, R3, R30, R31, R32, R33, R34, R35, R36, R37, R38, R39, R4, R40, R41, R48, R49, R5, R50, R51, R52, R53, R54, R55, R56, R57, R58, R59, R6, R60, R61, R62, R63, R64, R65, R66, R67, R68, R69, R7, R70, R71, R8, R9: footprint Resistor_SMD:R_0603_1608Metric -> Resistor_SMD:R_0402_1005Metric
- R100: value 10k -> 2k2; Note DNP -> (none); now left out of the parts list
- R101: value 1k -> 27R
- R102: value 470 -> 10k; Note (none) -> DNP; now not fitted
- R104: value 1k -> 220R
- R89: value 220 -> 1k
- R91: value 1K -> 1k
- R92: value 620R -> 75R
- R93: value 680k -> 75R
- R94: value 75 -> 75R
- R95: value 75 -> 620R
- R96: value 75 -> 680k
- R97: value 10k -> 1K
- R98: value 2k2 -> 1K
- R99: value 27R -> 10k
- TP10: value Luma -> Odd / Even
- TP4: value Composite Sync -> Composite
- TP5: value Vertical Sync -> Chroma
- TP6: value Horizontal Sync -> Luma
- TP7: value Odd / Even -> Composite Sync
- TP8: value Composite -> Vertical Sync
- TP9: value Chroma -> Horizontal Sync
- U1: value ICE40HX1K-VQ100 -> iCE40HX1K-VQ100
- renumbered C32 to C30, C30 to C31, C31 to C32, C35 to C37, C63 to C62, C64 to C63, C68 to C66, U14 to D10, U15 to D11, D3 to D4, D4 to D5, J3 to J2, J8 to J7, J9 to J8, J10 to J9, R112 to R114, R132 to R136, R133 to R137, R136 to R138, R88 to R90, U16 to U14, U17 to U15
Connections:
- net Audio Out is gone; now on net +1V1: C52.2
- net +1V1: no longer C45.2
- net +1V2: now also C65.2, C68.1, U16.5 (VOUT)
- net +3V3: now also C46.2, C51.1, R101.1, R102.1, R104.2, C64.2, D12.1 (A), R132.1, R133.1, U11.4 (VCC), U16.1 (VIN), U16.3 (EN); no longer C36.2, C48.1, C65.2, R100.1, R89.2, R97.1
- net +5V: now also C42.2, D2.1 (K), J3.1, J6.1 (VBUS), U10.8 (VCC); no longer C38.2, D2.5 (K), J1.7 (Pin_7)
- net 2354_SWCLK: now also J5.1 (Pin_1)
- net 2354_SWDIO: now also J5.3 (Pin_3)
- net 2354_USB_D+: now also J6.3 (D+)
- net 2354_USB_D-: now also J6.2 (D-)
- net 3V3.ADDRESS0: now also U14.16 (B7); no longer U14.22 (B1)
- net 3V3.ADDRESS1: now also U14.17 (B6); no longer U14.21 (B2)
- net 3V3.ADDRESS2: now also U14.18 (B5); no longer U14.20 (B3)
- net 3V3.ADDRESS4: now also U14.20 (B3); no longer U14.18 (B5)
- net 3V3.ADDRESS5: now also U14.21 (B2); no longer U14.17 (B6)
- net 3V3.CR_~{W}: now also U15.22 (B1); no longer U14.14 (B9)
- net 3V3.DATA0: now also U15.13 (B10); no longer U15.22 (B1)
- net 3V3.DATA1: now also U15.14 (B9); no longer U15.21 (B2)
- net 3V3.DATA2: now also U15.15 (B8); no longer U15.20 (B3)
- net 3V3.DATA3: now also U15.16 (B7); no longer U15.19 (B4)
- net 3V3.DATA4: now also U15.17 (B6); no longer U15.18 (B5)
- net 3V3.DATA5: now also U15.18 (B5); no longer U15.17 (B6)
- net 3V3.DATA6: now also U15.19 (B4); no longer U15.16 (B7)
- net 3V3.DATA7: now also U15.20 (B3); no longer U15.15 (B8)
- net 3V3.IO0: now also U15.21 (B2); no longer U14.15 (B8)
- net 3V3.SO2: now also U14.22 (B1); no longer U14.16 (B7)
- net 3V3_9110.CA1: now also U1.37 (IOB_37); no longer U1.29 (IOB_29)
- net 3V3_9110.CA2: now also U1.42 (IOB_43_CBSEL1); no longer U1.26 (IOB_26)
- net 3V3_9110.CB1: now also U1.36 (IOB_34); no longer U1.30 (IOB_30)
- net 3V3_9110.CB2: now also U1.41 (IOB_42_CBSEL0); no longer U1.27 (IOB_27)
- net 3V3_9110.~{NMI}: now also U1.40 (IOB_41); no longer U1.28 (IOB_28)
- net 3V3_9120.CA1: now also U1.30 (IOB_30); no longer U1.36 (IOB_34)
- net 3V3_9120.CA2: now also U1.28 (IOB_28); no longer U1.40 (IOB_41)
- net 3V3_9120.CB1: now also U1.29 (IOB_29); no longer U1.37 (IOB_37)
- net 3V3_9120.CB2: now also U1.27 (IOB_27); no longer U1.41 (IOB_42_CBSEL0)
- net 3V3_9120.~{IRQ}: now also U1.26 (IOB_26); no longer U1.42 (IOB_43_CBSEL1)
- net 5V_9110.CB1: now also D6.5 (IO4), D6.6 (NC)
- net 5V_9110.CB2: now also D8.5 (IO4), D8.6 (NC)
- net 5V_9110.PA2: now also D6.1 (IO1), D6.10 (NC)
- net 5V_9110.PA3: now also D3.5 (IO4), D3.6 (NC)
- net 5V_9110.PA4: now also D3.4 (IO3), D3.7 (NC)
- net 5V_9110.PA5: now also D3.2 (IO2), D3.9 (NC), J4.1 (Pin_1)
- net 5V_9110.PA6: now also D2.5 (K), D3.1 (IO1), D3.10 (NC); no longer D2.1 (K)
- net 5V_9110.PB0: now also D6.2 (IO2), D6.9 (NC)
- net 5V_9110.PB1: now also D7.1 (IO1), D7.10 (NC)
- net 5V_9110.PB2: now also D7.2 (IO2), D7.9 (NC)
- net 5V_9110.PB3: now also D7.4 (IO3), D7.7 (NC)
- net 5V_9110.PB4: now also D7.5 (IO4), D7.6 (NC)
- net 5V_9110.PB5: now also D8.1 (IO1), D8.10 (NC)
- net 5V_9110.PB6: now also D8.2 (IO2), D8.9 (NC)
- net 5V_9110.PB7: now also D8.4 (IO3), D8.7 (NC)
- net 5V_9120.CB1: now also D9.3 (K); no longer D9.1 (K)
- net 5V_9120.PB3: now also D2.4 (K); no longer D2.3 (K)
- net 9VAC~: now also AC1.1 (Pin_1); no longer BR1.3, C10.2, C12.1, FL1.2
- net BPOUT: now also TP9.1, U10.5 (BPOUT); no longer TP6.1
- net CASSETTE_READ: now also D2.3 (K); no longer D2.4 (K)
- net COMP_COLOUR: now also RV2.3, J4.8 (Pin_8); no longer RV1.3
- net COMP_SOUND: now also R89.1, C35.2, J4.2 (Pin_2); no longer C51.2, R103.1
- net EXT_AUDIO_IN: now also R91.2, J4.3 (Pin_3); no longer R104.2
- net GND: now also C34.1, C40.1, C48.1, C51.2, C52.1, R96.2, RV2.1, C35.1, C64.1, C68.2, D3.3 (G), D3.8 (G), D6.3 (G), D6.8 (G), D7.3 (G), D7.8 (G), D8.3 (G), D8.8 (G), J3.2, J5.2 (Pin_2), J6.5 (GND), J6.SH (Shield), R112.2, R88.1, U10.4 (GND), U11.5 (GND), U16.2 (GND); no longer C36.1, C41.1, C43.1, C48.2, C50.1, C51.1, J1.8 (Pin_8), R102.1, R93.2, RV1.1
- net IO.ADDRESS0: now also U14.8 (A7); no longer U14.2 (A1)
- net IO.ADDRESS1: now also U14.7 (A6); no longer U14.3 (A2)
- net IO.ADDRESS2: now also U14.6 (A5); no longer U14.4 (A3)
- net IO.ADDRESS4: now also U14.4 (A3); no longer U14.6 (A5)
- net IO.ADDRESS5: now also U14.3 (A2); no longer U14.7 (A6)
- net IO.CR_~{W}: now also U15.2 (A1); no longer U14.10 (A9)
- net IO.DATA0: now also U15.11 (A10); no longer U15.2 (A1)
- net IO.DATA1: now also U15.10 (A9); no longer U15.3 (A2)
- net IO.DATA2: now also U15.9 (A8); no longer U15.4 (A3)
- net IO.DATA3: now also U15.8 (A7); no longer U15.5 (A4)
- net IO.DATA4: now also U15.7 (A6); no longer U15.6 (A5)
- net IO.DATA5: now also U15.6 (A5); no longer U15.7 (A6)
- net IO.DATA6: now also U15.5 (A4); no longer U15.8 (A7)
- net IO.DATA7: now also U15.4 (A3); no longer U15.9 (A8)
- net IO.IO0: now also U15.3 (A2); no longer U14.9 (A8)
- net IO.SO2: now also U14.2 (A1); no longer U14.8 (A7)
- net POT_X: now also J4.5 (Pin_5)
- net POT_Y: now also J4.4 (Pin_4)
- net SERIAL_ATTN_IO: now also D9.1 (K); no longer D9.3 (K)
- net SERIAL_CLK_IO: now also D9.5 (K); no longer D9.4 (K)
- net SERIAL_DATA_IO: now also D9.4 (K); no longer D9.5 (K)
- net SYNC_LUMA: now also RV1.1, J4.7 (Pin_7); no longer RV2.1
- net VIC_CHROMA: now also R93.1, R98.1, U11.7 (CH.2_OUT); no longer R95.1
- net VIC_COMPOSITE: now also R92.1, U11.8 (CH.1_OUT); no longer R94.1
- net VIC_LUMA: now also R94.1, R97.1, U11.6 (CH.3_OUT); no longer R91.1, R96.1
- net VSOUT: now also TP8.1, U10.3 (VSOUT); no longer TP5.1
- net iCE40.DONE: now also R133.2
- net iCE40.~{RESET}: now also R132.2
- net ~{5V_RESET}: now also D6.4 (IO3), D6.7 (NC)
- net ~{CS}: now also R100.1, R102.2; no longer R100.2, R98.1
- net at C40.2: now also R96.1, U10.6 (RSET)
- net at R113.1: now also U14.14 (B9); no longer U15.14 (B9)
- net at S1.1, U13.26 (RUN): now also R99.2; no longer R97.2
- net at R134.1: now also U14.9 (A8); no longer U15.10 (A9)
- net at R135.1: now also U14.10 (A9); no longer U15.11 (A10)
- net at R95.2: now also C38.2, R94.2, TP6.1; no longer TP9.1
- net at C41.2: now also U10.2 (CVIN); no longer R93.1
- net at U13.21 (XIN), Y1.1: now also C44.2; no longer C43.2
- net at RV1.2: now also C50.2
- net at U1.75 (VPP_2V5): now also D12.3 (K)
- net at TP4.1: now also R92.2, J3.4, J3.5
- net at TP7.1: now also U10.1 (CSOUT)
- net at Je1.1 (Pin_1): now also R100.2; no longer R98.2
- net at R101.2: now also C48.2, U13.46 (VREG_AVDD); no longer U13.22 (XOUT)
- net at RV2.2: now also U11.2 (CH.2_IN); no longer C34.2
- net '9VAC~ renamed '9VAC22
- net '9VAC22: no longer EDGE2.11 (9V_AC_)
- new net: C45.2, R103.1, Y1.3
- new net: R93.2, TP5.1
- new net: C41.1, R95.1
- new net: R103.2, U13.22 (XOUT)
- new net: C43.1, U11.1 (CH.1_IN)
- new net: C50.1, U11.3 (CH.3_IN)
- new net: R112.1, U14.15 (B8)
- new net: TP10.1, U10.7 (OEOUT)
- new net: R104.1, RV1.3
- new net: C34.2, Q1.1 (B), R89.2, R91.1
- new net: C36.1, Q1.2 (E), R88.2
- new net: C43.2, R97.2, R98.2
- new net 9VAC22: BR1.3, C10.2, C12.1, FL1.2
- new net AUDIO OUT: C36.2, J3.3
- new net ~{9VAC~}: AC1.2 (Pin_2), EDGE2.11 (9V_AC_)
- no-connect marks 27 -> 28
Other:
- note removed: "FIRE"
- moved on the sheet: C30, C31, C62, D9, R18, R19, R20, R21, R22, R23, R24, R25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

Commit message: - Reorganised the prototype IO board layout for easier routing.
Parts:
- removed R112: 10k, Resistor_SMD:R_0603_1608Metric, symbol Device:R_Small
- added R149: 10k, Resistor_SMD:R_0603_1608Metric, symbol Device:R_Small
- C10, C11, C12, C9, FL1, SW1: now not fitted; now left out of the parts list
Connections:
- net 3V3.ADDRESS0: now also U1.100 (IOT_95), U14.15 (B8); no longer U1.78 (IOT_73), U14.16 (B7)
- net 3V3.ADDRESS1: now also U1.99 (IOT_93), U14.16 (B7); no longer U1.79 (IOT_74), U14.17 (B6)
- net 3V3.ADDRESS2: now also U1.97 (IOT_91), U14.17 (B6); no longer U1.80 (IOT_75), U14.18 (B5)
- net 3V3.ADDRESS3: now also U1.96 (IOT_90), U14.18 (B5); no longer U1.81 (IOT_77), U14.19 (B4)
- net 3V3.ADDRESS4: now also U1.95 (IOT_89), U14.19 (B4); no longer U1.82 (IOT_78), U14.20 (B3)
- net 3V3.ADDRESS5: now also U1.94 (IOT_88), U14.20 (B3); no longer U1.83 (IOT_79), U14.21 (B2)
- net 3V3.CR_~{W}: now also U14.22 (B1); no longer U15.22 (B1)
- net 3V3.DATA0: now also U1.86 (IOT_81); no longer U1.85 (IOT_80)
- net 3V3.DATA1: now also U1.85 (IOT_80); no longer U1.86 (IOT_81)
- net 3V3.DATA2: now also U1.83 (IOT_79); no longer U1.87 (IOT_82)
- net 3V3.DATA3: now also U1.82 (IOT_78); no longer U1.91 (IOT_86)
- net 3V3.DATA4: now also U1.81 (IOT_77); no longer U1.93 (IOT_87)
- net 3V3.DATA5: now also U1.80 (IOT_75); no longer U1.94 (IOT_88)
- net 3V3.DATA6: now also U1.79 (IOT_74); no longer U1.95 (IOT_89)
- net 3V3.DATA7: now also U1.78 (IOT_73); no longer U1.96 (IOT_90)
- net 3V3.IO0: now also R121.2, U14.21 (B2); no longer R122.2, U15.21 (B2)
- net 3V3.SO2: now also R122.2, U15.21 (B2); no longer R121.2, U14.22 (B1)
- net 3V3_9110.CA1: now also U1.36 (IOB_34); no longer U1.37 (IOB_37)
- net 3V3_9110.CB1: now also U1.41 (IOB_42_CBSEL0); no longer U1.36 (IOB_34)
- net 3V3_9110.CB2: now also U1.40 (IOB_41); no longer U1.41 (IOB_42_CBSEL0)
- net 3V3_9110.~{NMI}: now also U1.37 (IOB_37); no longer U1.40 (IOB_41)
- net 3V3_9120.CA1: now also U1.26 (IOB_26); no longer U1.30 (IOB_30)
- net 3V3_9120.CA2: now also U1.30 (IOB_30); no longer U1.28 (IOB_28)
- net 3V3_9120.CB2: now also U1.28 (IOB_28); no longer U1.27 (IOB_27)
- net 3V3_9120.~{IRQ}: now also U1.27 (IOB_27); no longer U1.26 (IOB_26)
- net GND: now also R134.1, R149.1; no longer R134.2
- net IO.ADDRESS0: now also U14.9 (A8); no longer U14.8 (A7)
- net IO.ADDRESS1: now also U14.8 (A7); no longer U14.7 (A6)
- net IO.ADDRESS2: now also U14.7 (A6); no longer U14.6 (A5)
- net IO.ADDRESS3: now also U14.6 (A5); no longer U14.5 (A4)
- net IO.ADDRESS4: now also U14.5 (A4); no longer U14.4 (A3)
- net IO.ADDRESS5: now also U14.4 (A3); no longer U14.3 (A2)
- net IO.CR_~{W}: now also U14.2 (A1); no longer U15.2 (A1)
- net IO.IO0: now also R121.1, U14.3 (A2); no longer R122.1, U15.3 (A2)
- net IO.SO2: now also R122.1, U15.3 (A2); no longer R121.1, U14.2 (A1)
- new net: R149.2, U15.2 (A1)
- new net: R134.2, U15.22 (B1)
Other:
- moved on the sheet: C63

Commit message: - Routed the new prototype 2 IO board.
Parts:
- removed D2: ESDA6V1SC5, _Custom:SOT-553, symbol Power_Protection:ESDA6V1SC5
- removed TP4: Composite, TestPoint:TestPoint_Pad_1.0x1.0mm, symbol Connector:TestPoint
- added AC2: 9VAC, Connector_PinHeader_2.54mm:PinHeader_1x02_P2.54mm_Vertical, symbol Connector:Conn_01x02_Pin
- added C71: 4.7uf, Capacitor_SMD:C_0603_1608Metric, symbol Device:C_Small
- added D13: ESDALD05UG4X, Package_SON:USON-10_2.5x1.0mm_P0.5mm, symbol Power_Protection:TPD4E02B04DQA
- added TP14: 9VAC_N, TestPoint:TestPoint_Pad_1.0x1.0mm, symbol Connector:TestPoint
- added TP15: 9VAC_L, TestPoint:TestPoint_Pad_1.0x1.0mm, symbol Connector:TestPoint
- JP1: value SolderJumper_2_Bridged -> CA2
- JP2: value SolderJumper_2_Bridged -> PA7
- JP3: value SolderJumper_2_Bridged -> PA0
- JP4: value SolderJumper_2_Bridged -> PA1
- R102: now left out of the parts list
- TP1: value TestPoint -> GBIn7
- TP2: value TestPoint -> GBin6
- renumbered C61 to C55, C55 to C61
Connections:
- net 9VAC is gone; now on net 9VAC_L: C11.2, FL1.1, SW1.1
- net +5V: now also D5.3 (K), D13.5 (IO4), D13.6 (NC); no longer D4.5 (K)
- net 3V3.CR_~{W}: now also R121.2, U1.90 (IOT_85_GBIN0), U14.21 (B2); no longer R123.2, U1.89 (IOT_84_GBIN1), U14.22 (B1)
- net 3V3.IO0: now also R123.2, U1.89 (IOT_84_GBIN1), U14.22 (B1); no longer R121.2, U1.90 (IOT_85_GBIN0), U14.21 (B2)
- net 3V3.SO2: now also U1.63 (IOR_61_GBIN2); no longer U1.62 (IOR_60_GBIN3)
- net 5V_9110.PA2: now also D5.1 (K); no longer D4.1 (K)
- net 5V_9110.PA3: now also D5.4 (K); no longer D5.5 (K)
- net 5V_9110.PA4: now also D4.1 (K); no longer D5.4 (K)
- net 5V_9110.PA5: now also D5.5 (K); no longer D5.1 (K)
- net 5V_9110.PA6: now also D13.1 (IO1), D13.10 (NC)
- net 5V_9120.CB1: now also D9.1 (K); no longer D9.3 (K)
- net 5V_9120.PB3: now also D13.2 (IO2), D13.9 (NC)
- net 5V_9120.PB7: now also D4.5 (K); no longer D5.3 (K)
- net CASSETTE_READ: now also D13.4 (IO3), D13.7 (NC)
- net CLK_25MHZ: now also U1.62 (IOR_60_GBIN3); no longer U1.63 (IOR_61_GBIN2)
- net GND: now also C71.1, D13.3 (G), D13.8 (G)
- net IO.CR_~{W}: now also R121.1, U14.3 (A2); no longer R123.1, U14.2 (A1)
- net IO.IO0: now also R123.1, U14.2 (A1); no longer R121.1, U14.3 (A2)
- net MOTOR_6VDC: now also C71.2
- net SERIAL_ATTN_IO: now also D9.3 (K); no longer D9.1 (K)
- net SERIAL_CLK_IO: now also D9.4 (K); no longer D9.5 (K)
- net SERIAL_DATA_IO: now also D9.5 (K); no longer D9.4 (K)
- net at C15.2, L1.2, SW1.4: now also DIN1.4, DIN1.5, SW1.5
- net 9VAC_L: now reaches DIN1.6, SW1.2
- net 9VAC_L: now also TP15.1
- net '9VAC renamed 9VAC_N
- net 9VAC_N: now also TP14.1
- net '9VAC22 renamed 9VAC_L2
- net 9VAC_L2: now also AC2.1 (Pin_1)
- net 9VAC22 renamed 9VAC_N2
- net 9VAC_N2: now also AC2.2 (Pin_2)
Other:
- note added: "AC supply hacked out of prototype. Only needed by user port."
- note added: "Remove Bridge"
- moved on the sheet: C32, C33, D4, U9
